Commit message: New eef, working scene loading, updated param loader

File: ros/tabletop_description/urdf/eef_macro.xacro (robot description, xacro)
@@ -12,5 +12,6 @@
       <visual>
         <geometry>
-          <sphere radius="${radius}" />
+          <mesh filename="package://tabletop_description/meshes/visual/eef.stl"
+            scale="0.001 0.001 0.001" />
         </geometry>
         <origin rpy="0 0 0" xyz="0 0 0" />
@@ -18,5 +19,5 @@
       <collision>
         <geometry>
-          <sphere radius="${radius}" />
+          <mesh filename="package://tabletop_description/meshes/collision/eef.stl" />
         </geometry>
         <origin rpy="0 0 0" xyz="0 0 0" />
@@ -25,7 +26,7 @@
         <mass value="${mass}" />
         <origin xyz="0 0 0" rpy="0 0 0" />
-        <inertia ixx="${(2/5) * mass * radius * radius}" ixy="0" ixz="0"
-          iyy="${(2/5) * mass * radius * radius}" iyz="0"
-          izz="${(2/5) * mass * radius * radius}" />
+        <inertia ixx="${(1/12) * mass * (3 * radius * radius)}" ixy="0" ixz="0"
+          iyy="${(1/12) * mass * (3 * radius * radius)}" iyz="0"
+          izz="${(1/2) * mass * radius * radius}" />
       </inertial>
     </link>

File: ros/tabletop_description/urdf/tabletop_macro.xacro (robot description, xacro)
@@ -35,14 +35,14 @@
       force_abs_paths="${force_abs_paths}"
     >
-      <origin xyz="0 0 0.05" rpy="0 0 ${pi/2.0}" />
+      <origin xyz="0 0 0.05" rpy="0 0 0" />
     </xacro:ur_robot>
     <!-- end effector -->
     <xacro:eef
       tf_prefix="${tf_prefix}"
-      parent="${tf_prefix}flange"
+      parent="${tf_prefix}wrist_3_link"
       radius="${eef_radius}"
       mass="${eef_mass}"
     >
-      <origin xyz="0 0 0" rpy="${pi/2.0} 0 ${pi/2.0}" />
+      <origin xyz="0 0 0.0315" rpy="${pi} 0 0" />
     </xacro:eef>
     <!-- scene -->

File: ros/tabletop_moveit_config/srdf/tabletop_macro.srdf.xacro (robot description, xacro)
@@ -25,9 +25,9 @@
     - Groups can also be formed by referencing to already defined group names-->
     <group name="ur_manipulator">
-      <chain base_link="base_link" tip_link="flange" />
+      <chain base_link="base_link" tip_link="eef" />
     </group>
-    <group name="ur_eef">
+    <!-- <group name="ur_eef">
       <link name="eef" />
-    </group>
+    </group> -->
     <!--GROUP
     STATES: Purpose: Define a named state for a particular group, in terms of joint values. This is
@@ -59,6 +59,6 @@
     <!--END
     EFFECTOR - Purpose - Represent information about an end effector.-->
-    <end_effector name="ur_eef" parent_link="flange" group="ur_eef"
-      parent_group="ur_manipulator" />
+    <!-- <end_effector name="ur_eef" parent_link="flange" group="ur_eef"
+      parent_group="ur_manipulator" /> -->
     <!--VIRTUAL
     JOINT - Purpose - this element defines a virtual joint between a robot link and an external

Commit message: Temp commit to compare to previous

File: ros/tabletop_description/urdf/eef_macro.xacro (robot description, xacro)
@@ -9,9 +9,8 @@
     mass
     ">
-    <link name="${tf_prefix}eef">
+    <link name="${tf_prefix}eef_link">
       <visual>
         <geometry>
-          <mesh filename="package://tabletop_description/meshes/visual/eef.stl"
-            scale="0.001 0.001 0.001" />
+          <mesh filename="package://tabletop_description/meshes/visual/eef.stl" />
         </geometry>
         <origin rpy="0 0 0" xyz="0 0 0" />
@@ -31,7 +30,14 @@
       </inertial>
     </link>
-    <joint name="${parent}-eef" type="fixed">
+    <joint name="${parent}-eef_link" type="fixed">
       <xacro:insert_block name="origin" />
       <parent link="${parent}" />
+      <child link="${tf_prefix}eef_link" />
+    </joint>
+    <!-- eef -->
+    <link name="${tf_prefix}eef" />
+    <joint name="${tf_prefix}eef_link-eef" type="fixed">
+      <xacro:insert_block name="origin" />
+      <parent link="${tf_prefix}eef_link" />
       <child link="${tf_prefix}eef" />
     </joint>

File: ros/tabletop_description/urdf/tabletop_macro.xacro (robot description, xacro)
@@ -44,5 +44,5 @@
       mass="${eef_mass}"
     >
-      <origin xyz="0 0 0.0315" rpy="${pi} 0 0" />
+      <origin xyz="0 0 -0.005" rpy="0 0 0" />
     </xacro:eef>
     <!-- scene -->

File: ros/tabletop_moveit_config/srdf/tabletop_macro.srdf.xacro (robot description, xacro)
@@ -34,7 +34,7 @@
     useful to define states like 'folded arms'-->
     <group_state name="erect" group="ur_manipulator">
+      <joint name="shoulder_pan_joint" value="0" />
+      <joint name="shoulder_lift_joint" value="${-pi/2}" />
       <joint name="elbow_joint" value="0" />
-      <joint name="shoulder_lift_joint" value="-1.5707" />
-      <joint name="shoulder_pan_joint" value="0" />
       <joint name="wrist_1_joint" value="0" />
       <joint name="wrist_2_joint" value="0" />
@@ -42,12 +42,20 @@
     </group_state>
     <group_state name="flaccid" group="ur_manipulator">
+      <joint name="shoulder_pan_joint" value="0" />
+      <joint name="shoulder_lift_joint" value="0" />
       <joint name="elbow_joint" value="0" />
-      <joint name="shoulder_lift_joint" value="0" />
-      <joint name="shoulder_pan_joint" value="0" />
       <joint name="wrist_1_joint" value="0" />
       <joint name="wrist_2_joint" value="0" />
       <joint name="wrist_3_joint" value="0" />
     </group_state>
-    <group_state name="test_configuration" group="ur_manipulator">
+    <group_state name="semi" group="ur_manipulator">
+      <joint name="shoulder_pan_joint" value="0" />
+      <joint name="shoulder_lift_joint" value="${-pi/2}" />
+      <joint name="elbow_joint" value="${pi/2}" />
+      <joint name="wrist_1_joint" value="0" />
+      <joint name="wrist_2_joint" value="0" />
+      <joint name="wrist_3_joint" value="0" />
+    </group_state>
+    <group_state name="test" group="ur_manipulator">
       <joint name="elbow_joint" value="1.4" />
       <joint name="shoulder_lift_joint" value="-1.62" />
@@ -70,9 +78,8 @@
     collision with any other link in the robot. This tag disables collision checking between a
     specified pair of links. -->
-    <!-- <disable_collisions link1="base_link" link2="scene" reason="Adjacent" /> -->
     <disable_collisions link1="base_link_inertia" link2="shoulder_link" reason="Adjacent" />
-    <disable_collisions link1="eef" link2="wrist_1_link" reason="Never" />
-    <disable_collisions link1="eef" link2="wrist_2_link" reason="Default" />
-    <disable_collisions link1="eef" link2="wrist_3_link" reason="Adjacent" />
+    <disable_collisions link1="eef_link" link2="wrist_1_link" reason="Never" />
+    <disable_collisions link1="eef_link" link2="wrist_2_link" reason="Default" />
+    <disable_collisions link1="eef_link" link2="wrist_3_link" reason="Adjacent" />
     <disable_collisions link1="forearm_link" link2="upper_arm_link" reason="Adjacent" />
     <disable_collisions link1="forearm_link" link2="wrist_1_link" reason="Adjacent" />

Commit message: Temp commit to save moveit_config before modifying

File: ros/tabletop_description/urdf/eef_macro.xacro (robot description, xacro)
@@ -1,4 +1,5 @@
 <?xml version="1.0"?>
 <robot xmlns:xacro="http://ros.org/wiki/xacro">
+  <xacro:include filename="$(find tabletop_description)/urdf/sphere_macro.xacro" />
   <xacro:macro name="eef"
     params="
@@ -6,7 +7,10 @@
     parent
     *origin
-    radius
-    mass
     ">
+    <xacro:property name="length" value="0.0365" />
+    <xacro:property name="radius" value="0.0315" />
+    <xacro:property name="mass" value="0.5" />
+    <xacro:property name="sphere_radius" value="0.05" />
+    <xacro:property name="sphere_mass" value="0.01" />
     <link name="${tf_prefix}eef_link">
       <visual>
@@ -14,5 +18,5 @@
           <mesh filename="package://tabletop_description/meshes/visual/eef.stl" />
         </geometry>
-        <origin rpy="0 0 0" xyz="0 0 0" />
+        <origin xyz="0 0 0" rpy="0 0 0" />
       </visual>
       <collision>
@@ -20,14 +24,22 @@
           <mesh filename="package://tabletop_description/meshes/collision/eef.stl" />
         </geometry>
-        <origin rpy="0 0 0" xyz="0 0 0" />
+        <origin xyz="0 0 0" rpy="0 0 0" />
       </collision>
       <inertial>
         <mass value="${mass}" />
-        <origin xyz="0 0 0" rpy="0 0 0" />
-        <inertia ixx="${(1/12) * mass * (3 * radius * radius)}" ixy="0" ixz="0"
-          iyy="${(1/12) * mass * (3 * radius * radius)}" iyz="0"
-          izz="${(1/2) * mass * radius * radius}" />
+        <origin xyz="0 0 ${length/2}" rpy="0 0 0" />
+        <inertia ixx="${mass * (3 * radius * radius + length * length) / 12}" ixy="0" ixz="0"
+          iyy="${mass * (3 * radius * radius + length * length) / 12}" iyz="0"
+          izz="${mass * radius * radius / 2}" />
       </inertial>
     </link>
+    <xacro:sphere
+      tf_prefix="${tf_prefix}"
+      parent="${parent}"
+      radius="${sphere_radius}"
+      mass="${sphere_mass}"
+    >
+      <xacro:insert_block name="origin" />
+    </xacro:sphere>
     <joint name="${parent}-eef_link" type="fixed">
       <xacro:insert_block name="origin" />
@@ -35,8 +47,10 @@
       <child link="${tf_prefix}eef_link" />
     </joint>
-    <!-- eef -->
+    <!-- eef frame, X+ direction to move to attach object,
+         Y+ left,
+         Z+ up / outward from eef -->
     <link name="${tf_prefix}eef" />
     <joint name="${tf_prefix}eef_link-eef" type="fixed">
-      <xacro:insert_block name="origin" />
+      <origin xyz="0 0 ${length}" rpy="0 0 ${pi/2}" />
       <parent link="${tf_prefix}eef_link" />
       <child link="${tf_prefix}eef" />

File: ros/tabletop_description/urdf/sphere_macro.xacro (robot description, xacro)
@@ -1,7 +1,8 @@
 <?xml version="1.0"?>
 <robot xmlns:xacro="http://ros.org/wiki/xacro">
-  <xacro:macro name="eef"
+  <xacro:macro name="sphere"
     params="
     tf_prefix
+    name
     parent
     *origin
@@ -9,5 +10,5 @@
     mass
     ">
-    <link name="${tf_prefix}eef">
+    <link name="${tf_prefix}${name}">
       <visual>
         <geometry>
@@ -30,8 +31,8 @@
       </inertial>
     </link>
-    <joint name="${parent}-eef" type="fixed">
+    <joint name="${parent}-${name}" type="fixed">
       <xacro:insert_block name="origin" />
       <parent link="${parent}" />
-      <child link="${tf_prefix}eef" />
+      <child link="${tf_prefix}${name}" />
     </joint>
   </xacro:macro>

File: ros/tabletop_description/urdf/tabletop.urdf.xacro (robot description, xacro)
@@ -22,6 +22,4 @@
   <xacro:arg name="safety_k_position" default="20" />
   <xacro:arg name="force_abs_paths" default="false" />
-  <xacro:arg name="eef_radius" default="0.06" />
-  <xacro:arg name="eef_mass" default="0.5" />
   <!-- tabletop -->
   <xacro:tabletop
@@ -36,6 +34,4 @@
     safety_k_position="$(arg safety_k_position)"
     force_abs_paths="$(arg force_abs_paths)"
-    eef_radius="$(arg eef_radius)"
-    eef_mass="$(arg eef_mass)"
   />
 </robot>

File: ros/tabletop_description/urdf/tabletop_control.urdf.xacro (robot description, xacro)
@@ -54,7 +54,4 @@
     default="$(find ur_description)/config/initial_positions.yaml" />
   <xacro:property name="initial_positions_file" default="$(arg initial_positions_file)" />
-  <!-- end effector parameters -->
-  <xacro:arg name="eef_radius" default="0.06" />
-  <xacro:arg name="eef_mass" default="0.5" />
   <!-- tabletop -->
   <xacro:tabletop
@@ -69,6 +66,4 @@
     safety_k_position="$(arg safety_k_position)"
     force_abs_paths="$(arg force_abs_paths)"
-    eef_radius="$(arg eef_radius)"
-    eef_mass="$(arg eef_mass)"
   />
   <xacro:ur_ros2_control

File: ros/tabletop_description/urdf/tabletop_macro.xacro (robot description, xacro)
@@ -16,7 +16,9 @@
     safety_k_position
     force_abs_paths
-    eef_radius
-    eef_mass
     ">
+    <xacro:property name="robot_offset_xyz" value="0 0 0.05" />
+    <xacro:property name="robot_offset_rpy" value="0 0 ${pi/2}" />
+    <xacro:property name="eef_offset_xyz" value="0 0 -0.005" />
+    <xacro:property name="eef_offset_rpy" value="0 0 0" />
     <!-- world -->
     <link name="world" />
@@ -35,5 +37,5 @@
       force_abs_paths="${force_abs_paths}"
     >
-      <origin xyz="0 0 0.05" rpy="0 0 0" />
+      <origin xyz="${robot_offset_xyz}" rpy="${robot_offset_rpy}" />
     </xacro:ur_robot>
     <!-- end effector -->
@@ -41,8 +43,6 @@
       tf_prefix="${tf_prefix}"
       parent="${tf_prefix}wrist_3_link"
-      radius="${eef_radius}"
-      mass="${eef_mass}"
     >
-      <origin xyz="0 0 -0.005" rpy="0 0 0" />
+      <origin xyz="${eef_offset_xyz}" rpy="${eef_offset_rpy}" />
     </xacro:eef>
     <!-- scene -->

Commit message: Planning around objects in updated planning scene with collision objects, error with rviz materials

File: ros/tabletop_description/urdf/eef_macro.xacro (robot description, xacro)
@@ -11,5 +11,5 @@
     <xacro:property name="radius" value="0.0315" />
     <xacro:property name="mass" value="0.5" />
-    <xacro:property name="sphere_radius" value="0.05" />
+    <xacro:property name="sphere_radius" value="0.06" />
     <xacro:property name="sphere_mass" value="0.01" />
     <link name="${tf_prefix}eef_link">

File: ros/tabletop_description/urdf/sphere_macro.xacro (robot description, xacro)
@@ -4,5 +4,4 @@
     params="
     tf_prefix
-    name
     parent
     *origin
@@ -10,5 +9,5 @@
     mass
     ">
-    <link name="${tf_prefix}${name}">
+    <link name="${tf_prefix}sphere">
       <visual>
         <geometry>
@@ -31,8 +30,8 @@
       </inertial>
     </link>
-    <joint name="${parent}-${name}" type="fixed">
+    <joint name="${parent}-sphere" type="fixed">
       <xacro:insert_block name="origin" />
       <parent link="${parent}" />
-      <child link="${tf_prefix}${name}" />
+      <child link="${tf_prefix}sphere" />
     </joint>
   </xacro:macro>

File: ros/tabletop_moveit_config/srdf/tabletop_macro.srdf.xacro (robot description, xacro)
@@ -79,7 +79,4 @@
     specified pair of links. -->
     <disable_collisions link1="base_link_inertia" link2="shoulder_link" reason="Adjacent" />
-    <disable_collisions link1="eef_link" link2="wrist_1_link" reason="Never" />
-    <disable_collisions link1="eef_link" link2="wrist_2_link" reason="Default" />
-    <disable_collisions link1="eef_link" link2="wrist_3_link" reason="Adjacent" />
     <disable_collisions link1="forearm_link" link2="upper_arm_link" reason="Adjacent" />
     <disable_collisions link1="forearm_link" link2="wrist_1_link" reason="Adjacent" />
@@ -89,4 +86,11 @@
     <disable_collisions link1="wrist_1_link" link2="wrist_3_link" reason="Never" />
     <disable_collisions link1="wrist_2_link" link2="wrist_3_link" reason="Adjacent" />
+    <disable_collisions link1="eef_link" link2="wrist_1_link" reason="Never" />
+    <disable_collisions link1="eef_link" link2="wrist_2_link" reason="Default" />
+    <disable_collisions link1="eef_link" link2="wrist_3_link" reason="Adjacent" />
+    <disable_collisions link1="sphere" link2="wrist_1_link" reason="Never" />
+    <disable_collisions link1="sphere" link2="wrist_2_link" reason="Default" />
+    <disable_collisions link1="sphere" link2="wrist_3_link" reason="Adjacent" />
+    <disable_collisions link1="sphere" link2="eef_link" reason="Adjacent" />
   </xacro:macro>
 </robot>
