Commit message: Updated fetch/return logic and config, integrated task code and tested using simple task

File: ros/tabletop_description/urdf/sphere_macro.xacro (robot description, xacro)
@@ -10,10 +10,4 @@
     ">
     <link name="${tf_prefix}sphere">
-      <visual>
-        <geometry>
-          <sphere radius="${radius}" />
-        </geometry>
-        <origin rpy="0 0 0" xyz="0 0 0" />
-      </visual>
       <collision>
         <geometry>
@@ -22,11 +16,4 @@
         <origin rpy="0 0 0" xyz="0 0 0" />
       </collision>
-      <inertial>
-        <mass value="${mass}" />
-        <origin xyz="0 0 0" rpy="0 0 0" />
-        <inertia ixx="${(2/5) * mass * radius * radius}" ixy="0" ixz="0"
-          iyy="${(2/5) * mass * radius * radius}" iyz="0"
-          izz="${(2/5) * mass * radius * radius}" />
-      </inertial>
     </link>
     <joint name="${parent}-sphere" type="fixed">
