Commit message: Who needs fusion (also robot working in new rig)

File: ros/tabletop_description/urdf/tabletop_control.urdf.xacro (robot description, xacro)
@@ -52,5 +52,5 @@
   <!-- initial position for simulations (Mock Hardware, Gazebo, Ignition) -->
   <xacro:arg name="initial_positions_file"
-    default="$(find ur_description)/config/initial_positions.yaml" />
+    default="$(find tabletop_description)/config/initial_positions.yaml" />
   <xacro:property name="initial_positions_file" default="$(arg initial_positions_file)" />
   <!-- tabletop -->

File: ros/tabletop_description/urdf/tabletop_macro.xacro (robot description, xacro)
@@ -3,5 +3,4 @@
   <xacro:include filename="$(find ur_description)/urdf/ur_macro.xacro" />
   <xacro:include filename="$(find tabletop_description)/urdf/eef_macro.xacro" />
-  <xacro:include filename="$(find tabletop_description)/urdf/scene_macro.xacro" />
   <xacro:macro name="tabletop"
     params="
@@ -17,6 +16,6 @@
     force_abs_paths
     ">
-    <xacro:property name="robot_offset_xyz" value="0 0 0.04" />
-    <xacro:property name="robot_offset_rpy" value="0 0 -1.5707" />
+    <xacro:property name="robot_offset_xyz" value="1.2143 1.1178 0.309" />
+    <xacro:property name="robot_offset_rpy" value="0 0 0" />
     <xacro:property name="eef_offset_xyz" value="0 0 -0.005" />
     <xacro:property name="eef_offset_rpy" value="0 0 0" />

File: ros/tabletop_moveit_config/srdf/tabletop_macro.srdf.xacro (robot description, xacro)
@@ -56,5 +56,5 @@
       <joint name="shoulder_lift_joint" value="${-pi/2}" />
       <joint name="elbow_joint" value="${pi/2}" />
-      <joint name="wrist_1_joint" value="0" />
+      <joint name="wrist_1_joint" value="${-pi/2}" />
       <joint name="wrist_2_joint" value="0" />
       <joint name="wrist_3_joint" value="0" />
