Commit message: Partially added examples to tabletop_tasks for asyncio usage

File: ros/tabletop_description/urdf/tabletop_macro.xacro (robot description, xacro)
@@ -47,11 +47,11 @@
     </xacro:eef>
     <!-- scene -->
-    <xacro:scene
+    <!-- <xacro:scene
       tf_prefix="${tf_prefix}"
       parent="world"
     >
       <origin xyz="0 0 0" rpy="0 0 0" />
-      <!-- <origin xyz="0.843 -0.891 0.85886" rpy="0 0 0" /> -->
-    </xacro:scene>
+    </xacro:scene> -->
+    <!-- <origin xyz="0.843 -0.891 0.85886" rpy="0 0 0" /> -->
   </xacro:macro>
 </robot>

Commit message: Static and dynamic meshes loaded as collision objects with configurable paths, scaling, and individual poses

File: ros/tabletop_description/urdf/tabletop_macro.xacro (robot description, xacro)
@@ -35,5 +35,5 @@
       force_abs_paths="${force_abs_paths}"
     >
-      <origin xyz="0 0 0" rpy="0 0 ${pi/2.0}" />
+      <origin xyz="0 0 0.05" rpy="0 0 ${pi/2.0}" />
     </xacro:ur_robot>
     <!-- end effector -->

Commit message: Real-world test with simple rig loaded, compatibility with no-gil moveit_py planning implemented and tested

File: ros/tabletop_description/urdf/tabletop_macro.xacro (robot description, xacro)
@@ -17,5 +17,5 @@
     force_abs_paths
     ">
-    <xacro:property name="robot_offset_xyz" value="0 0 0.05" />
+    <xacro:property name="robot_offset_xyz" value="0 0 0.045" />
     <xacro:property name="robot_offset_rpy" value="0 0 ${pi/2}" />
     <xacro:property name="eef_offset_xyz" value="0 0 -0.005" />

Commit message: Simlulation working on rig computer. Updated shebangs for executables Modified velocity and acceleration scaling factors

File: ros/tabletop_description/urdf/tabletop_macro.xacro (robot description, xacro)
@@ -17,5 +17,5 @@
     force_abs_paths
     ">
-    <xacro:property name="robot_offset_xyz" value="0 0 0.045" />
+    <xacro:property name="robot_offset_xyz" value="0 0 0.04" />
     <xacro:property name="robot_offset_rpy" value="0 0 ${pi/2}" />
     <xacro:property name="eef_offset_xyz" value="0 0 -0.005" />

Commit message: To the robot, I am god, for I have given it both life and purpose

File: ros/tabletop_description/urdf/tabletop_macro.xacro (robot description, xacro)
@@ -18,5 +18,5 @@
     ">
     <xacro:property name="robot_offset_xyz" value="0 0 0.04" />
-    <xacro:property name="robot_offset_rpy" value="0 0 ${pi/2}" />
+    <xacro:property name="robot_offset_rpy" value="0 0 -1.5707" />
     <xacro:property name="eef_offset_xyz" value="0 0 -0.005" />
     <xacro:property name="eef_offset_rpy" value="0 0 0" />

Commit message: I'm actually fuzzed up rn

File: ros/tabletop_description/urdf/tabletop_macro.xacro (robot description, xacro)
@@ -16,5 +16,5 @@
     force_abs_paths
     ">
-    <xacro:property name="robot_offset_xyz" value="1.2143 1.1178 0.309" />
+    <xacro:property name="robot_offset_xyz" value="1.247 1.0832 0.2685" />
     <xacro:property name="robot_offset_rpy" value="0 0 0" />
     <xacro:property name="eef_offset_xyz" value="0 0 -0.005" />

Commit message: Fuzziness inbound, I promise this time (also new small objects, simplified rig model, huge planning scene and fetching returning pipeline refactor, you wouldn't even believe

File: ros/tabletop_description/urdf/tabletop_macro.xacro (robot description, xacro)
@@ -16,5 +16,5 @@
     force_abs_paths
     ">
-    <xacro:property name="robot_offset_xyz" value="1.247 1.0832 0.2685" />
+    <xacro:property name="robot_offset_xyz" value="1.2468 1.0832 0.2685" />
     <xacro:property name="robot_offset_rpy" value="0 0 0" />
     <xacro:property name="eef_offset_xyz" value="0 0 -0.005" />

File: ros/tabletop_moveit_config/srdf/tabletop_macro.srdf.xacro (robot description, xacro)
@@ -68,4 +68,12 @@
       <joint name="wrist_3_joint" value="-0.11" />
     </group_state>
+    <group_state name="ready_for_action" group="ur_manipulator">
+      <joint name="shoulder_pan_joint" value="${pi/2}" />
+      <joint name="shoulder_lift_joint" value="${-pi/6}" />
+      <joint name="elbow_joint" value="${-2*pi/3}" />
+      <joint name="wrist_1_joint" value="${-2*pi/3}" />
+      <joint name="wrist_2_joint" value="${-pi/2}" />
+      <joint name="wrist_3_joint" value="${pi}" />
+    </group_state>
     <!--END
     EFFECTOR - Purpose - Represent information about an end effector.-->
@@ -75,6 +83,5 @@
     JOINT - Purpose - this element defines a virtual joint between a robot link and an external
     frame of reference (considered fixed with respect to the robot)-->
-    <virtual_joint name="virtual_joint" type="fixed" parent_frame="world"
-      child_link="base_link" />
+    <virtual_joint name="virtual_joint" type="fixed" parent_frame="world" child_link="base_link" />
     <!--DISABLE
     COLLISIONS - By default it is assumed that any link of the robot could potentially come into

Commit message: Running (sort of) on real rig

File: ros/tabletop_description/urdf/tabletop_macro.xacro (robot description, xacro)
@@ -16,11 +16,14 @@
     force_abs_paths
     ">
-    <xacro:property name="robot_offset_xyz" value="1.2468 1.0832 0.2685" />
-    <xacro:property name="robot_offset_rpy" value="0 0 0" />
+    <!-- <xacro:property name="robot_offset_xyz" value="1.2468 1.0832 0.2685" /> -->
+    <!-- <xacro:property name="robot_offset_xyz" value="1.2482 1.0588 0.3342" /> -->
+    <!-- <xacro:property name="robot_offset_xyz" value="1.247 1.1279 0.309" /> -->
+    <xacro:property name="robot_offset_xyz" value="1.2504 1.0625 0.3085" />
+    <xacro:property name="robot_offset_rpy" value="0 0 -1.5707" />
     <xacro:property name="eef_offset_xyz" value="0 0 -0.005" />
     <xacro:property name="eef_offset_rpy" value="0 0 0" />
     <!-- world -->
     <link name="world" />
-    <!-- arm -->
+    <!-- robot -->
     <xacro:ur_robot
       name="${name}"
@@ -45,12 +48,4 @@
       <origin xyz="${eef_offset_xyz}" rpy="${eef_offset_rpy}" />
     </xacro:eef>
-    <!-- scene -->
-    <!-- <xacro:scene
-      tf_prefix="${tf_prefix}"
-      parent="world"
-    >
-      <origin xyz="0 0 0" rpy="0 0 0" />
-    </xacro:scene> -->
-    <!-- <origin xyz="0.843 -0.891 0.85886" rpy="0 0 0" /> -->
   </xacro:macro>
 </robot>

File: ros/tabletop_moveit_config/srdf/tabletop_macro.srdf.xacro (robot description, xacro)
@@ -27,10 +27,4 @@
       <chain base_link="base_link" tip_link="eef" />
     </group>
-    <group name="ur_wrist_2">
-      <chain base_link="base_link" tip_link="wrist_2_link" />
-    </group>
-    <!-- <group name="ur_eef">
-      <link name="eef" />
-    </group> -->
     <!--GROUP
     STATES: Purpose: Define a named state for a particular group, in terms of joint values. This is
@@ -69,5 +63,5 @@
     </group_state>
     <group_state name="ready_for_action" group="ur_manipulator">
-      <joint name="shoulder_pan_joint" value="${-pi/2}" />
+      <joint name="shoulder_pan_joint" value="0" />
       <joint name="shoulder_lift_joint" value="${-5*pi/6}" />
       <joint name="elbow_joint" value="${2*pi/3}" />
@@ -76,8 +70,4 @@
       <joint name="wrist_3_joint" value="${pi}" />
     </group_state>
-    <!--END
-    EFFECTOR - Purpose - Represent information about an end effector.-->
-    <!-- <end_effector name="ur_eef" parent_link="flange" group="ur_eef"
-      parent_group="ur_manipulator" /> -->
     <!--VIRTUAL
     JOINT - Purpose - this element defines a virtual joint between a robot link and an external
