Commit message: Added smoothing, fixed some small errors in detaching the object, refactored bin directory

File: ros/tabletop_description/urdf/cylinder_macro.xacro (robot description, xacro)
@@ -1,5 +1,5 @@
-<?xml version="1.0"?>
-<robot xmlns:xacro="http://ros.org/wiki/xacro">
-  <xacro:macro name="sphere"
+<?xml version="1.0" encoding="utf-8"?>
+<robot xmlns:xacro="http://www.ros.org/wiki/xacro">
+  <xacro:macro name="cylinder"
     params="
     name
@@ -8,11 +8,12 @@
     *origin
     radius
+    length
     ">
     <link name="${tf_prefix}${name}">
       <collision>
         <geometry>
-          <sphere radius="${radius}" />
+          <cylinder radius="${radius}" length="${length}" />
         </geometry>
-        <origin rpy="0 0 0" xyz="0 0 0" />
+        <origin xyz="0 0 ${length/2}" rpy="0 0 0" />
       </collision>
     </link>

File: ros/tabletop_description/urdf/eef_macro.xacro (robot description, xacro)
@@ -2,4 +2,5 @@
 <robot xmlns:xacro="http://ros.org/wiki/xacro">
   <xacro:include filename="$(find tabletop_description)/urdf/sphere_macro.xacro" />
+  <xacro:include filename="$(find tabletop_description)/urdf/cylinder_macro.xacro" />
   <xacro:macro name="eef"
     params="
@@ -12,5 +13,6 @@
     <xacro:property name="mass" value="0.5" />
     <xacro:property name="sphere_radius" value="0.06" />
-    <xacro:property name="sphere_mass" value="0.01" />
+    <xacro:property name="bounding_cylinder_radius" value="0.05" />
+    <xacro:property name="bounding_cylinder_length" value="0.11" />
     <link name="${tf_prefix}eef_link">
       <visual>
@@ -19,10 +21,13 @@
         </geometry>
         <origin xyz="0 0 0" rpy="0 0 0" />
+        <material name="black">
+          <color rgba="0 0 0 1" />
+        </material>
       </visual>
       <collision>
         <geometry>
-          <mesh filename="package://tabletop_description/meshes/collision/eef.stl" />
+          <cylinder radius="${radius}" length="${length}" />
         </geometry>
-        <origin xyz="0 0 0" rpy="0 0 0" />
+        <origin xyz="0 0 ${length/2}" rpy="0 0 0" />
       </collision>
       <inertial>
@@ -35,8 +40,8 @@
     </link>
     <xacro:sphere
+      name="eef_sphere"
       tf_prefix="${tf_prefix}"
       parent="${parent}"
       radius="${sphere_radius}"
-      mass="${sphere_mass}"
     >
       <xacro:insert_block name="origin" />
@@ -56,4 +61,13 @@
       <child link="${tf_prefix}eef" />
     </joint>
+    <!-- <xacro:cylinder
+      name="bounding_cylinder"
+      tf_prefix="${tf_prefix}"
+      parent="${tf_prefix}eef"
+      radius="${bounding_cylinder_radius}"
+      length="${bounding_cylinder_length}"
+    >
+      <origin xyz="0 0 0" rpy="0 0 0" />
+    </xacro:cylinder> -->
   </xacro:macro>
 </robot>

File: ros/tabletop_moveit_config/srdf/tabletop_macro.srdf.xacro (robot description, xacro)
@@ -79,5 +79,7 @@
     specified pair of links. -->
     <disable_collisions link1="base_link_inertia" link2="shoulder_link" reason="Adjacent" />
-    <disable_collisions link1="eef_link" link2="sphere" reason="Default" />
+    <disable_collisions link1="eef_link" link2="eef_sphere" reason="Default" />
+    <!-- <disable_collisions link1="eef_link" link2="bounding_cylinder" reason="Default" />
+    <disable_collisions link1="bounding_cylinder" link2="eef_sphere" reason="Default" /> -->
     <disable_collisions link1="eef_link" link2="wrist_1_link" reason="Never" />
     <disable_collisions link1="eef_link" link2="wrist_2_link" reason="Never" />
@@ -87,7 +89,10 @@
     <disable_collisions link1="forearm_link" link2="wrist_2_link" reason="Never" />
     <disable_collisions link1="shoulder_link" link2="upper_arm_link" reason="Adjacent" />
-    <disable_collisions link1="sphere" link2="wrist_1_link" reason="Never" />
-    <disable_collisions link1="sphere" link2="wrist_2_link" reason="Default" />
-    <disable_collisions link1="sphere" link2="wrist_3_link" reason="Adjacent" />
+    <disable_collisions link1="eef_sphere" link2="wrist_1_link" reason="Never" />
+    <disable_collisions link1="eef_sphere" link2="wrist_2_link" reason="Default" />
+    <disable_collisions link1="eef_sphere" link2="wrist_3_link" reason="Adjacent" />
+    <!-- <disable_collisions link1="bounding_cylinder" link2="wrist_1_link" reason="Never" />
+    <disable_collisions link1="bounding_cylinder" link2="wrist_2_link" reason="Default" />
+    <disable_collisions link1="bounding_cylinder" link2="wrist_3_link" reason="Adjacent" /> -->
     <disable_collisions link1="wrist_1_link" link2="wrist_2_link" reason="Adjacent" />
     <disable_collisions link1="wrist_1_link" link2="wrist_3_link" reason="Never" />
