Commit message: Added eef tool, tcp_pose_broadcaster seems to be interfering/overwriting /robot_description topic

File: ros/tabletop_description/urdf/tabletop.urdf.xacro (robot description, xacro)
@@ -1,26 +1,55 @@
 <?xml version="1.0"?>
-<robot name="tabletop" xmlns:xacro="http://ros.org/wiki/xacro">
-    <xacro:include filename="$(find tabletop_description)/urdf/tabletop_macro.xacro" />
-    <xacro:arg name="ur_type" default="ur5e" />
-    <xacro:arg name="joint_limits_parameters_file"
-        default="$(find ur_description)/config/$(arg ur_type)/joint_limits.yaml" />
-    <xacro:arg name="kinematics_parameters_file"
-        default="$(find ur_description)/config/$(arg ur_type)/default_kinematics.yaml" />
-    <xacro:arg name="physical_parameters_file"
-        default="$(find ur_description)/config/$(arg ur_type)/physical_parameters.yaml" />
-    <xacro:arg name="visual_parameters_file"
-        default="$(find ur_description)/config/$(arg ur_type)/visual_parameters.yaml" />
-    <link name="world" />
-    <!--This
-  will create the scene where the robot is located in-->
-    <xacro:tabletop
-        parent="world"
-        ur_type="$(arg ur_type)"
-        joint_limits_parameters_file="$(arg joint_limits_parameters_file)"
-        kinematics_parameters_file="$(arg kinematics_parameters_file)"
-        physical_parameters_file="$(arg physical_parameters_file)"
-        visual_parameters_file="$(arg visual_parameters_file)"
-    >
-        <origin xyz="0 0 1" rpy="0 0 0" />
-    </xacro:tabletop>
+<robot xmlns:xacro="http://wiki.ros.org/xacro" name="$(arg name)">
+  <!-- robot name parameter -->
+  <xacro:arg name="name" default="ur" />
+  <!-- Include eef and ur description-->
+  <xacro:include filename="$(find ur_description)/urdf/ur_macro.xacro" />
+  <xacro:include filename="$(find tabletop_description)/urdf/tabletop_eef_macro.xacro" />
+  <!-- possible 'ur_type' values: ur3, ur3e, ur5, ur5e, ur10, ur10e, ur16e, ur20, ur30 -->
+  <!-- the default value should raise an error in case this was called without defining the type -->
+  <xacro:arg name="ur_type" default="ur5x" />
+  <!-- parameters -->
+  <xacro:arg name="tf_prefix" default="" />
+  <xacro:arg name="joint_limit_params"
+    default="$(find ur_description)/config/$(arg ur_type)/joint_limits.yaml" />
+  <xacro:arg name="kinematics_params"
+    default="$(find ur_description)/config/$(arg ur_type)/default_kinematics.yaml" />
+  <xacro:arg name="physical_params"
+    default="$(find ur_description)/config/$(arg ur_type)/physical_parameters.yaml" />
+  <xacro:arg name="visual_params"
+    default="$(find ur_description)/config/$(arg ur_type)/visual_parameters.yaml" />
+  <xacro:arg name="transmission_hw_interface" default="" />
+  <xacro:arg name="safety_limits" default="false" />
+  <xacro:arg name="safety_pos_margin" default="0.15" />
+  <xacro:arg name="safety_k_position" default="20" />
+  <!--When
+  using gazebo simulations absolute paths are necessary.-->
+  <xacro:arg name="force_abs_paths" default="false" />
+  <!-- create link fixed to the "world" -->
+  <link name="world" />
+  <!-- arm -->
+  <xacro:ur_robot
+    name="$(arg name)"
+    tf_prefix="$(arg tf_prefix)"
+    parent="world"
+    joint_limits_parameters_file="$(arg joint_limit_params)"
+    kinematics_parameters_file="$(arg kinematics_params)"
+    physical_parameters_file="$(arg physical_params)"
+    visual_parameters_file="$(arg visual_params)"
+    safety_limits="$(arg safety_limits)"
+    safety_pos_margin="$(arg safety_pos_margin)"
+    safety_k_position="$(arg safety_k_position)"
+    force_abs_paths="$(arg force_abs_paths)"
+  >
+    <origin xyz="0 0 0" rpy="0 0 0" />          <!-- position robot in the world -->
+  </xacro:ur_robot>
+  <!-- end effector -->
+  <xacro:eef
+    tf_prefix="$(arg tf_prefix)"
+    parent="$(arg tf_prefix)flange"
+    radius="0.05"
+    mass="0.5"
+  >
+    <origin xyz="0 0 0" rpy="0 0 0" />
+  </xacro:eef>
 </robot>

File: ros/tabletop_moveit_config/srdf/tabletop.srdf.xacro (robot description, xacro)
@@ -3,5 +3,5 @@
   <!-- robot name parameter -->
   <xacro:arg name="name" default="ur" />
-  <xacro:include filename="$(find tabletop_moveit_config)/srdf/ur_macro.srdf.xacro" />
+  <xacro:include filename="$(find tabletop_moveit_config)/srdf/tabletop_macro.srdf.xacro" />
   <xacro:ur_srdf />
 </robot>

File: ros/tabletop_moveit_config/srdf/tabletop_macro.srdf.xacro (robot description, xacro)
@@ -7,5 +7,5 @@
   are defined
 -->
-  <xacro:macro name="ur_srdf" params="">
+  <xacro:macro name="ur_srdf">
     <!--GROUPS
     - Representation of a set of joints and links. This can be useful for specifying DOF to plan
@@ -27,8 +27,11 @@
       <chain base_link="base_link" tip_link="tool0" />
     </group>
+    <!-- <group name="ur_eef">
+      <link name="eef" />
+    </group> -->
     <!--GROUP
-    STATES - Purpose - Define a named state for a particular group, in terms of joint values. This
-    is useful to define states like 'folded arms'-->
-    <group_state name="home" group="ur_manipulator">
+    STATES: Purpose: Define a named state for a particular group, in terms of joint values. This is
+    useful to define states like 'folded arms'-->
+    <group_state name="erect" group="ur_manipulator">
       <joint name="elbow_joint" value="0" />
       <joint name="shoulder_lift_joint" value="-1.5707" />
@@ -38,9 +41,9 @@
       <joint name="wrist_3_joint" value="0" />
     </group_state>
-    <group_state name="up" group="ur_manipulator">
+    <group_state name="flaccid" group="ur_manipulator">
       <joint name="elbow_joint" value="0" />
-      <joint name="shoulder_lift_joint" value="-1.5707" />
+      <joint name="shoulder_lift_joint" value="0" />
       <joint name="shoulder_pan_joint" value="0" />
-      <joint name="wrist_1_joint" value="-1.5707" />
+      <joint name="wrist_1_joint" value="0" />
       <joint name="wrist_2_joint" value="0" />
       <joint name="wrist_3_joint" value="0" />
@@ -56,12 +59,16 @@
     <!--END
     EFFECTOR - Purpose - Represent information about an end effector.-->
+    <!-- <end_effector name="ur_eef" parent_link="flange" group="ur_eef"
+    parent_group="ur_manipulator" /> -->
     <!--VIRTUAL
     JOINT - Purpose - this element defines a virtual joint between a robot link and an external
     frame of reference (considered fixed with respect to the robot)-->
+    <!-- <virtual_joint name="virtual_joint" type="fixed" parent_frame="world"
+    child_link="base_link" /> -->
     <!--DISABLE
     COLLISIONS - By default it is assumed that any link of the robot could potentially come into
     collision with any other link in the robot. This tag disables collision checking between a
     specified pair of links. -->
-    <disable_collisions link1="base_link" link2="base_link_inertia" reason="Adjacent" />
+    <!-- <disable_collisions link1="base_link" link2="base_link_inertia" reason="Adjacent" />
     <disable_collisions link1="base_link_inertia" link2="shoulder_link" reason="Adjacent" />
     <disable_collisions link1="tool0" link2="wrist_1_link" reason="Never" />
@@ -73,4 +80,15 @@
     <disable_collisions link1="wrist_1_link" link2="wrist_2_link" reason="Adjacent" />
     <disable_collisions link1="wrist_1_link" link2="wrist_3_link" reason="Never" />
+    <disable_collisions link1="wrist_2_link" link2="wrist_3_link" reason="Adjacent" /> -->
+    <disable_collisions link1="base_link_inertia" link2="shoulder_link" reason="Adjacent" />
+    <disable_collisions link1="eef" link2="wrist_1_link" reason="Never" />
+    <disable_collisions link1="eef" link2="wrist_2_link" reason="Default" />
+    <disable_collisions link1="eef" link2="wrist_3_link" reason="Adjacent" />
+    <disable_collisions link1="forearm_link" link2="upper_arm_link" reason="Adjacent" />
+    <disable_collisions link1="forearm_link" link2="wrist_1_link" reason="Adjacent" />
+    <disable_collisions link1="forearm_link" link2="wrist_2_link" reason="Never" />
+    <disable_collisions link1="shoulder_link" link2="upper_arm_link" reason="Adjacent" />
+    <disable_collisions link1="wrist_1_link" link2="wrist_2_link" reason="Adjacent" />
+    <disable_collisions link1="wrist_1_link" link2="wrist_3_link" reason="Never" />
     <disable_collisions link1="wrist_2_link" link2="wrist_3_link" reason="Adjacent" />
   </xacro:macro>

Commit message: Added end effector link to urdf to prevent robot safety mechanism from going off

File: ros/tabletop_description/urdf/tabletop.urdf.xacro (robot description, xacro)
@@ -40,5 +40,4 @@
     safety_pos_margin="$(arg safety_pos_margin)"
     safety_k_position="$(arg safety_k_position)"
-    force_abs_paths="$(arg force_abs_paths)"
   >
     <origin xyz="0 0 0" rpy="0 0 0" />          <!-- position robot in the world -->

File: ros/tabletop_description/urdf/tabletop_control.urdf.xacro (robot description, xacro)
@@ -75,9 +75,9 @@
   <xacro:eef
     tf_prefix="$(arg tf_prefix)"
-    parent="$(arg tf_prefix)tool0"
+    parent="$(arg tf_prefix)flange"
     radius="0.05"
     mass="0.5"
   >
-    <origin xyz="0 0 0" rpy="0 0 0" />
+    <origin xyz="0 0 0" rpy="${pi/2.0} 0 ${pi/2.0}" />
   </xacro:eef>
   <xacro:ur_ros2_control

File: ros/tabletop_moveit_config/srdf/tabletop_macro.srdf.xacro (robot description, xacro)
@@ -25,9 +25,9 @@
     - Groups can also be formed by referencing to already defined group names-->
     <group name="ur_manipulator">
-      <chain base_link="base_link" tip_link="tool0" />
+      <chain base_link="base_link" tip_link="flange" />
     </group>
-    <!-- <group name="ur_eef">
+    <group name="ur_eef">
       <link name="eef" />
-    </group> -->
+    </group>
     <!--GROUP
     STATES: Purpose: Define a named state for a particular group, in terms of joint values. This is
@@ -59,26 +59,15 @@
     <!--END
     EFFECTOR - Purpose - Represent information about an end effector.-->
-    <!-- <end_effector name="ur_eef" parent_link="flange" group="ur_eef"
-    parent_group="ur_manipulator" /> -->
+    <end_effector name="ur_eef" parent_link="flange" group="ur_eef"
+      parent_group="ur_manipulator" />
     <!--VIRTUAL
     JOINT - Purpose - this element defines a virtual joint between a robot link and an external
     frame of reference (considered fixed with respect to the robot)-->
-    <!-- <virtual_joint name="virtual_joint" type="fixed" parent_frame="world"
-    child_link="base_link" /> -->
+    <virtual_joint name="virtual_joint" type="fixed" parent_frame="world"
+      child_link="base_link" />
     <!--DISABLE
     COLLISIONS - By default it is assumed that any link of the robot could potentially come into
     collision with any other link in the robot. This tag disables collision checking between a
     specified pair of links. -->
-    <!-- <disable_collisions link1="base_link" link2="base_link_inertia" reason="Adjacent" />
-    <disable_collisions link1="base_link_inertia" link2="shoulder_link" reason="Adjacent" />
-    <disable_collisions link1="tool0" link2="wrist_1_link" reason="Never" />
-    <disable_collisions link1="tool0" link2="wrist_2_link" reason="Never" />
-    <disable_collisions link1="tool0" link2="wrist_3_link" reason="Adjacent" />
-    <disable_collisions link1="forearm_link" link2="upper_arm_link" reason="Adjacent" />
-    <disable_collisions link1="forearm_link" link2="wrist_1_link" reason="Adjacent" />
-    <disable_collisions link1="shoulder_link" link2="upper_arm_link" reason="Adjacent" />
-    <disable_collisions link1="wrist_1_link" link2="wrist_2_link" reason="Adjacent" />
-    <disable_collisions link1="wrist_1_link" link2="wrist_3_link" reason="Never" />
-    <disable_collisions link1="wrist_2_link" link2="wrist_3_link" reason="Adjacent" /> -->
     <disable_collisions link1="base_link_inertia" link2="shoulder_link" reason="Adjacent" />
     <disable_collisions link1="eef" link2="wrist_1_link" reason="Never" />

Commit message: Added scene.dae file to URDF, planning with collision avoidance working, added x11 support as extended docker compose services, added custom rsp launch file and modularized urdf macros, reformatted .env files and added convenience scripts

File: ros/tabletop_description/urdf/tabletop.urdf.xacro (robot description, xacro)
@@ -4,9 +4,8 @@
   <xacro:arg name="name" default="ur" />
   <!-- Include eef and ur description-->
-  <xacro:include filename="$(find ur_description)/urdf/ur_macro.xacro" />
-  <xacro:include filename="$(find tabletop_description)/urdf/tabletop_eef_macro.xacro" />
+  <xacro:include filename="$(find tabletop_description)/urdf/tabletop_macro.xacro" />
   <!-- possible 'ur_type' values: ur3, ur3e, ur5, ur5e, ur10, ur10e, ur16e, ur20, ur30 -->
   <!-- the default value should raise an error in case this was called without defining the type -->
-  <xacro:arg name="ur_type" default="ur5x" />
+  <xacro:arg name="ur_type" default="urX" />
   <!-- parameters -->
   <xacro:arg name="tf_prefix" default="" />
@@ -19,18 +18,14 @@
   <xacro:arg name="visual_params"
     default="$(find ur_description)/config/$(arg ur_type)/visual_parameters.yaml" />
-  <xacro:arg name="transmission_hw_interface" default="" />
   <xacro:arg name="safety_limits" default="false" />
   <xacro:arg name="safety_pos_margin" default="0.15" />
   <xacro:arg name="safety_k_position" default="20" />
-  <!--When
-  using gazebo simulations absolute paths are necessary.-->
   <xacro:arg name="force_abs_paths" default="false" />
-  <!-- create link fixed to the "world" -->
-  <link name="world" />
-  <!-- arm -->
-  <xacro:ur_robot
+  <xacro:arg name="eef_radius" default="0.06" />
+  <xacro:arg name="eef_mass" default="0.5" />
+  <!-- tabletop -->
+  <xacro:tabletop
     name="$(arg name)"
     tf_prefix="$(arg tf_prefix)"
-    parent="world"
     joint_limits_parameters_file="$(arg joint_limit_params)"
     kinematics_parameters_file="$(arg kinematics_params)"
@@ -40,15 +35,7 @@
     safety_pos_margin="$(arg safety_pos_margin)"
     safety_k_position="$(arg safety_k_position)"
-  >
-    <origin xyz="0 0 0" rpy="0 0 0" />          <!-- position robot in the world -->
-  </xacro:ur_robot>
-  <!-- end effector -->
-  <xacro:eef
-    tf_prefix="$(arg tf_prefix)"
-    parent="$(arg tf_prefix)flange"
-    radius="0.05"
-    mass="0.5"
-  >
-    <origin xyz="0 0 0" rpy="0 0 0" />
-  </xacro:eef>
+    force_abs_paths="$(arg force_abs_paths)"
+    eef_radius="$(arg eef_radius)"
+    eef_mass="$(arg eef_mass)"
+  />
 </robot>

File: ros/tabletop_description/urdf/tabletop_control.urdf.xacro (robot description, xacro)
@@ -2,13 +2,12 @@
 <robot xmlns:xacro="http://wiki.ros.org/xacro" name="$(arg name)">
   <!-- robot name parameter -->
-  <xacro:arg name="name" default="ur5e" />
+  <xacro:arg name="name" default="ur" />
   <!-- Include eef and ur description-->
-  <xacro:include filename="$(find ur_description)/urdf/ur_macro.xacro" />
-  <xacro:include filename="$(find tabletop_description)/urdf/tabletop_eef_macro.xacro" />
+  <xacro:include filename="$(find tabletop_description)/urdf/tabletop_macro.xacro" />
   <xacro:include filename="$(find ur_robot_driver)/urdf/ur.ros2_control.xacro" />
   <xacro:include filename="$(find ur_description)/urdf/inc/ur_transmissions.xacro" />
   <!-- possible 'ur_type' values: ur3, ur3e, ur5, ur5e, ur10, ur10e, ur16e, ur20 -->
   <!-- the default value should raise an error in case this was called without defining the type -->
-  <xacro:arg name="ur_type" default="ur5e" />
+  <xacro:arg name="ur_type" default="urX" />
   <!-- parameters -->
   <xacro:arg name="tf_prefix" default="" />
@@ -25,4 +24,5 @@
   <xacro:arg name="safety_pos_margin" default="0.15" />
   <xacro:arg name="safety_k_position" default="20" />
+  <xacro:arg name="force_abs_paths" default="false" />
   <!-- ros2_control related parameters -->
   <xacro:arg name="headless_mode" default="false" />
@@ -53,13 +53,12 @@
   <xacro:arg name="initial_positions_file"
     default="$(find ur_description)/config/initial_positions.yaml" />
-  <!-- convert to property to use substitution in function -->
   <xacro:property name="initial_positions_file" default="$(arg initial_positions_file)" />
-  <!-- create link fixed to the "world" -->
-  <link name="world" />
-  <!-- arm -->
-  <xacro:ur_robot
+  <!-- end effector parameters -->
+  <xacro:arg name="eef_radius" default="0.06" />
+  <xacro:arg name="eef_mass" default="0.5" />
+  <!-- tabletop -->
+  <xacro:tabletop
     name="$(arg name)"
     tf_prefix="$(arg tf_prefix)"
-    parent="world"
     joint_limits_parameters_file="$(arg joint_limit_params)"
     kinematics_parameters_file="$(arg kinematics_params)"
@@ -69,16 +68,8 @@
     safety_pos_margin="$(arg safety_pos_margin)"
     safety_k_position="$(arg safety_k_position)"
-  >
-    <origin xyz="0 0 0" rpy="0 0 0" />          <!-- position robot in the world -->
-  </xacro:ur_robot>
-  <!-- end effector -->
-  <xacro:eef
-    tf_prefix="$(arg tf_prefix)"
-    parent="$(arg tf_prefix)flange"
-    radius="0.05"
-    mass="0.5"
-  >
-    <origin xyz="0 0 0" rpy="${pi/2.0} 0 ${pi/2.0}" />
-  </xacro:eef>
+    force_abs_paths="$(arg force_abs_paths)"
+    eef_radius="$(arg eef_radius)"
+    eef_mass="$(arg eef_mass)"
+  />
   <xacro:ur_ros2_control
     name="$(arg name)"

File: ros/tabletop_moveit_config/srdf/tabletop_macro.srdf.xacro (robot description, xacro)
@@ -70,4 +70,5 @@
     collision with any other link in the robot. This tag disables collision checking between a
     specified pair of links. -->
+    <disable_collisions link1="base_link" link2="scene" reason="Adjacent" />
     <disable_collisions link1="base_link_inertia" link2="shoulder_link" reason="Adjacent" />
     <disable_collisions link1="eef" link2="wrist_1_link" reason="Never" />
