Commit message: New and improved nonsense, should work exactly like before

File: ros/tabletop_description/urdf/tabletop.urdf.xacro (robot description, xacro)
@@ -5,5 +5,7 @@
   <!-- Include eef and ur description-->
   <xacro:include filename="$(find tabletop_description)/urdf/tabletop_macro.xacro" />
-  <!-- possible 'ur_type' values: ur3, ur3e, ur5, ur5e, ur10, ur10e, ur16e, ur20, ur30 -->
+  <xacro:include filename="$(find ur_robot_driver)/urdf/ur.ros2_control.xacro" />
+  <xacro:include filename="$(find ur_description)/urdf/inc/ur_transmissions.xacro" />
+  <!-- possible 'ur_type' values: ur3, ur3e, ur5, ur5e, ur10, ur10e, ur16e, ur20 -->
   <!-- the default value should raise an error in case this was called without defining the type -->
   <xacro:arg name="ur_type" default="urX" />
@@ -18,8 +20,38 @@
   <xacro:arg name="visual_params"
     default="$(find ur_description)/config/$(arg ur_type)/visual_parameters.yaml" />
+  <xacro:arg name="transmission_hw_interface" default="" />
   <xacro:arg name="safety_limits" default="false" />
   <xacro:arg name="safety_pos_margin" default="0.15" />
   <xacro:arg name="safety_k_position" default="20" />
   <xacro:arg name="force_abs_paths" default="false" />
+  <!-- ros2_control related parameters -->
+  <xacro:arg name="headless_mode" default="false" />
+  <xacro:arg name="robot_ip" default="0.0.0.0" />
+  <xacro:arg name="script_filename" default="" />
+  <xacro:arg name="output_recipe_filename" default="" />
+  <xacro:arg name="input_recipe_filename" default="" />
+  <xacro:arg name="reverse_ip" default="0.0.0.0" />
+  <xacro:arg name="script_command_port" default="50004" />
+  <xacro:arg name="reverse_port" default="50001" />
+  <xacro:arg name="script_sender_port" default="50002" />
+  <xacro:arg name="trajectory_port" default="50003" />
+  <!--   tool communication related parameters-->
+  <xacro:arg name="use_tool_communication" default="false" />
+  <xacro:arg name="tool_voltage" default="0" />
+  <xacro:arg name="tool_parity" default="0" />
+  <xacro:arg name="tool_baud_rate" default="115200" />
+  <xacro:arg name="tool_stop_bits" default="1" />
+  <xacro:arg name="tool_rx_idle_chars" default="1.5" />
+  <xacro:arg name="tool_tx_idle_chars" default="3.5" />
+  <xacro:arg name="tool_device_name" default="/tmp/ttyUR" />
+  <xacro:arg name="tool_tcp_port" default="54321" />
+  <!-- Simulation parameters -->
+  <xacro:arg name="use_mock_hardware" default="false" />
+  <xacro:arg name="mock_sensor_commands" default="false" />
+  <xacro:arg name="simulation_controllers" default="" />
+  <!-- initial position for simulations (Mock Hardware, Gazebo, Ignition) -->
+  <xacro:arg name="initial_positions_file"
+    default="$(find tabletop_description)/config/initial_positions.yaml" />
+  <xacro:property name="initial_positions_file" default="$(arg initial_positions_file)" />
   <!-- tabletop -->
   <xacro:tabletop
@@ -35,3 +67,31 @@
     force_abs_paths="$(arg force_abs_paths)"
   />
+  <xacro:ur_ros2_control
+    name="$(arg name)"
+    tf_prefix="$(arg tf_prefix)"
+    kinematics_parameters_file="$(arg kinematics_params)"
+    transmission_hw_interface="$(arg transmission_hw_interface)"
+    use_mock_hardware="$(arg use_mock_hardware)"
+    mock_sensor_commands="$(arg mock_sensor_commands)"
+    headless_mode="$(arg headless_mode)"
+    initial_positions="${xacro.load_yaml(initial_positions_file)}"
+    use_tool_communication="$(arg use_tool_communication)"
+    tool_voltage="$(arg tool_voltage)"
+    tool_parity="$(arg tool_parity)"
+    tool_baud_rate="$(arg tool_baud_rate)"
+    tool_stop_bits="$(arg tool_stop_bits)"
+    tool_rx_idle_chars="$(arg tool_rx_idle_chars)"
+    tool_tx_idle_chars="$(arg tool_tx_idle_chars)"
+    tool_device_name="$(arg tool_device_name)"
+    tool_tcp_port="$(arg tool_tcp_port)"
+    robot_ip="$(arg robot_ip)"
+    script_filename="$(arg script_filename)"
+    output_recipe_filename="$(arg output_recipe_filename)"
+    input_recipe_filename="$(arg input_recipe_filename)"
+    reverse_ip="$(arg reverse_ip)"
+    script_command_port="$(arg script_command_port)"
+    reverse_port="$(arg reverse_port)"
+    script_sender_port="$(arg script_sender_port)"
+    trajectory_port="$(arg trajectory_port)"
+  />
 </robot>

File: ros/tabletop_moveit_config/srdf/tabletop_macro.srdf.xacro (robot description, xacro)
@@ -24,5 +24,5 @@
     <!--SUBGROUPS
     - Groups can also be formed by referencing to already defined group names-->
-    <group name="ur_manipulator">
+    <group name="manipulator">
       <chain base_link="base_link" tip_link="eef" />
     </group>
@@ -30,5 +30,5 @@
     STATES: Purpose: Define a named state for a particular group, in terms of joint values. This is
     useful to define states like 'folded arms'-->
-    <group_state name="erect" group="ur_manipulator">
+    <group_state name="erect" group="manipulator">
       <joint name="shoulder_pan_joint" value="0" />
       <joint name="shoulder_lift_joint" value="${-pi/2}" />
@@ -38,5 +38,5 @@
       <joint name="wrist_3_joint" value="0" />
     </group_state>
-    <group_state name="flaccid" group="ur_manipulator">
+    <group_state name="flaccid" group="manipulator">
       <joint name="shoulder_pan_joint" value="0" />
       <joint name="shoulder_lift_joint" value="0" />
@@ -46,5 +46,5 @@
       <joint name="wrist_3_joint" value="0" />
     </group_state>
-    <group_state name="semi" group="ur_manipulator">
+    <group_state name="semi" group="manipulator">
       <joint name="shoulder_pan_joint" value="0" />
       <joint name="shoulder_lift_joint" value="${-pi/2}" />
@@ -54,5 +54,5 @@
       <joint name="wrist_3_joint" value="0" />
     </group_state>
-    <group_state name="ready_for_action" group="ur_manipulator">
+    <group_state name="ready_for_action" group="manipulator">
       <joint name="shoulder_pan_joint" value="0" />
       <joint name="shoulder_lift_joint" value="${-5*pi/6}" />
@@ -62,5 +62,5 @@
       <joint name="wrist_3_joint" value="${pi}" />
     </group_state>
-    <group_state name="pre_present" group="ur_manipulator">
+    <group_state name="pre_present" group="manipulator">
       <joint name="shoulder_pan_joint" value="-0.6065" />
       <joint name="shoulder_lift_joint" value="-0.6788" />
