Commit message: Fuzzing complete: - Fuzzy trajectory caching finally seems to work - Upgraded to sqlite3 for cache - Commander refactor: * Planning pipeline now accepts initialized planning component and request parameters * Fetch and return processes refactored to improve error handling and real robot recovery * Context manager improved * Thread pool executor increased max workers for faster trajectory planning/execution

File: ros/tabletop_moveit_config/srdf/tabletop_macro.srdf.xacro (robot description, xacro)
@@ -69,9 +69,9 @@
     </group_state>
     <group_state name="ready_for_action" group="ur_manipulator">
-      <joint name="shoulder_pan_joint" value="${pi/2}" />
-      <joint name="shoulder_lift_joint" value="${-pi/6}" />
-      <joint name="elbow_joint" value="${-2*pi/3}" />
-      <joint name="wrist_1_joint" value="${-2*pi/3}" />
-      <joint name="wrist_2_joint" value="${-pi/2}" />
+      <joint name="shoulder_pan_joint" value="${-pi/2}" />
+      <joint name="shoulder_lift_joint" value="${-5*pi/6}" />
+      <joint name="elbow_joint" value="${2*pi/3}" />
+      <joint name="wrist_1_joint" value="${-pi/3}" />
+      <joint name="wrist_2_joint" value="${pi/2}" />
       <joint name="wrist_3_joint" value="${pi}" />
     </group_state>

Commit message: Real robot working (except for 7,2 for some reason)

File: ros/tabletop_moveit_config/srdf/tabletop_macro.srdf.xacro (robot description, xacro)
@@ -54,12 +54,4 @@
       <joint name="wrist_3_joint" value="0" />
     </group_state>
-    <group_state name="test" group="ur_manipulator">
-      <joint name="elbow_joint" value="1.4" />
-      <joint name="shoulder_lift_joint" value="-1.62" />
-      <joint name="shoulder_pan_joint" value="1.54" />
-      <joint name="wrist_1_joint" value="-1.2" />
-      <joint name="wrist_2_joint" value="-1.6" />
-      <joint name="wrist_3_joint" value="-0.11" />
-    </group_state>
     <group_state name="ready_for_action" group="ur_manipulator">
       <joint name="shoulder_pan_joint" value="0" />
@@ -69,4 +61,12 @@
       <joint name="wrist_2_joint" value="${pi/2}" />
       <joint name="wrist_3_joint" value="${pi}" />
+    </group_state>
+    <group_state name="pre_present" group="ur_manipulator">
+      <joint name="shoulder_pan_joint" value="-0.6065" />
+      <joint name="shoulder_lift_joint" value="-0.6788" />
+      <joint name="elbow_joint" value="1.4381" />
+      <joint name="wrist_1_joint" value="-2.3351" />
+      <joint name="wrist_2_joint" value="1.5686" />
+      <joint name="wrist_3_joint" value="3.7411" />
     </group_state>
     <!--VIRTUAL
