Commit message: Absolutely blasting through testing
- Dashboard interface wildly improved
- Robot base and object mount poses recalibrated
- Dummy task for dummy easy testing
- Various qol features
- Real robot fixes/changes
- Foraging vastly improved
- Future workload increased twofold

File: src/ros/tabletop/tabletop_description/urdf/tabletop_macro.xacro (robot description, xacro)
@@ -19,5 +19,6 @@
     <!-- <xacro:property name="robot_offset_xyz" value="1.2482 1.0588 0.3342" /> -->
     <!-- <xacro:property name="robot_offset_xyz" value="1.247 1.1279 0.309" /> -->
-    <xacro:property name="robot_offset_xyz" value="1.2504 1.0625 0.3085" />
+    <!-- <xacro:property name="robot_offset_xyz" value="1.2504 1.0625 0.3085" /> -->
+    <xacro:property name="robot_offset_xyz" value="1.2554 1.0625 0.3085" />
     <xacro:property name="robot_offset_rpy" value="0 0 -1.5707" />
     <xacro:property name="eef_offset_xyz" value="0 0 -0.005" />
