Commit message: It's working, but it's slow af

File: src/ros/tabletop/tabletop_description/urdf/eef_macro.xacro (robot description, xacro)
@@ -13,6 +13,6 @@
     <xacro:property name="mass" value="0.5" />
     <xacro:property name="sphere_radius" value="0.06" />
-    <xacro:property name="bounding_cylinder_radius" value="0.05" />
-    <xacro:property name="bounding_cylinder_length" value="0.11" />
+    <!-- <xacro:property name="bounding_cylinder_radius" value="0.05" />
+    <xacro:property name="bounding_cylinder_length" value="0.11" /> -->
     <link name="${tf_prefix}eef_link">
       <visual>

File: src/ros/tabletop/tabletop_moveit_config/srdf/tabletop_macro.srdf.xacro (robot description, xacro)
@@ -79,23 +79,23 @@
     specified pair of links. -->
     <disable_collisions link1="base_link_inertia" link2="shoulder_link" reason="Adjacent" />
-    <disable_collisions link1="eef_link" link2="eef_sphere" reason="Default" />
+    <disable_collisions link1="shoulder_link" link2="upper_arm_link" reason="Adjacent" />
+    <disable_collisions link1="upper_arm_link" link2="forearm_link" reason="Adjacent" />
+    <disable_collisions link1="forearm_link" link2="wrist_1_link" reason="Adjacent" />
+    <disable_collisions link1="forearm_link" link2="wrist_2_link" reason="Never" />
+    <disable_collisions link1="wrist_1_link" link2="wrist_2_link" reason="Adjacent" />
+    <disable_collisions link1="wrist_1_link" link2="wrist_3_link" reason="Never" />
+    <disable_collisions link1="wrist_1_link" link2="eef_link" reason="Never" />
+    <disable_collisions link1="wrist_1_link" link2="eef_sphere" reason="Never" />
+    <disable_collisions link1="wrist_2_link" link2="wrist_3_link" reason="Adjacent" />
+    <disable_collisions link1="wrist_2_link" link2="eef_link" reason="Never" />
+    <disable_collisions link1="wrist_2_link" link2="eef_sphere" reason="Never" />
+    <disable_collisions link1="wrist_3_link" link2="eef_link" reason="Adjacent" />
+    <disable_collisions link1="wrist_3_link" link2="eef_sphere" reason="Adjacent" />
+    <disable_collisions link1="eef_link" link2="eef_sphere" reason="Adjacent" />
     <!-- <disable_collisions link1="eef_link" link2="bounding_cylinder" reason="Default" />
     <disable_collisions link1="bounding_cylinder" link2="eef_sphere" reason="Default" /> -->
-    <disable_collisions link1="eef_link" link2="wrist_1_link" reason="Never" />
-    <disable_collisions link1="eef_link" link2="wrist_2_link" reason="Never" />
-    <disable_collisions link1="eef_link" link2="wrist_3_link" reason="Adjacent" />
-    <disable_collisions link1="forearm_link" link2="upper_arm_link" reason="Adjacent" />
-    <disable_collisions link1="forearm_link" link2="wrist_1_link" reason="Adjacent" />
-    <disable_collisions link1="forearm_link" link2="wrist_2_link" reason="Never" />
-    <disable_collisions link1="shoulder_link" link2="upper_arm_link" reason="Adjacent" />
-    <disable_collisions link1="eef_sphere" link2="wrist_1_link" reason="Never" />
-    <disable_collisions link1="eef_sphere" link2="wrist_2_link" reason="Default" />
-    <disable_collisions link1="eef_sphere" link2="wrist_3_link" reason="Adjacent" />
     <!-- <disable_collisions link1="bounding_cylinder" link2="wrist_1_link" reason="Never" />
     <disable_collisions link1="bounding_cylinder" link2="wrist_2_link" reason="Default" />
     <disable_collisions link1="bounding_cylinder" link2="wrist_3_link" reason="Adjacent" /> -->
-    <disable_collisions link1="wrist_1_link" link2="wrist_2_link" reason="Adjacent" />
-    <disable_collisions link1="wrist_1_link" link2="wrist_3_link" reason="Never" />
-    <disable_collisions link1="wrist_2_link" link2="wrist_3_link" reason="Adjacent" />
   </xacro:macro>
 </robot>

Commit message: as branch name suggests

File: src/ros/tabletop/tabletop_description/urdf/eef_macro.xacro (robot description, xacro)
@@ -8,11 +8,9 @@
     parent
     *origin
+    cylinder_length
+    cylinder_radius
+    cylinder_mass
+    sphere_radius
     ">
-    <xacro:property name="length" value="0.0365" />
-    <xacro:property name="radius" value="0.0315" />
-    <xacro:property name="mass" value="0.5" />
-    <xacro:property name="sphere_radius" value="0.06" />
-    <!-- <xacro:property name="bounding_cylinder_radius" value="0.05" />
-    <xacro:property name="bounding_cylinder_length" value="0.11" /> -->
     <link name="${tf_prefix}eef_link">
       <visual>
@@ -27,14 +25,17 @@
       <collision>
         <geometry>
-          <cylinder radius="${radius}" length="${length}" />
+          <cylinder radius="${cylinder_radius}" length="${cylinder_length}" />
         </geometry>
-        <origin xyz="0 0 ${length/2}" rpy="0 0 0" />
+        <origin xyz="0 0 ${cylinder_length/2}" rpy="0 0 0" />
       </collision>
       <inertial>
-        <mass value="${mass}" />
-        <origin xyz="0 0 ${length/2}" rpy="0 0 0" />
-        <inertia ixx="${mass * (3 * radius * radius + length * length) / 12}" ixy="0" ixz="0"
-          iyy="${mass * (3 * radius * radius + length * length) / 12}" iyz="0"
-          izz="${mass * radius * radius / 2}" />
+        <mass value="${cylinder_mass}" />
+        <origin xyz="0 0 ${cylinder_length/2}" rpy="0 0 0" />
+        <inertia
+          ixx="${cylinder_mass * (3 * cylinder_radius * cylinder_radius + cylinder_length * cylinder_length) / 12}"
+          ixy="0" ixz="0"
+          iyy="${cylinder_mass * (3 * cylinder_radius * cylinder_radius + cylinder_length * cylinder_length) / 12}"
+          iyz="0"
+          izz="${cylinder_mass * cylinder_radius * cylinder_radius / 2}" />
       </inertial>
     </link>
@@ -57,5 +58,5 @@
     <link name="${tf_prefix}eef" />
     <joint name="${tf_prefix}eef_link-eef" type="fixed">
-      <origin xyz="0 0 ${length}" rpy="0 0 ${pi/2}" />
+      <origin xyz="0 0 ${cylinder_length}" rpy="0 0 ${pi/2}" />
       <parent link="${tf_prefix}eef_link" />
       <child link="${tf_prefix}eef" />

File: src/ros/tabletop/tabletop_description/urdf/tabletop.urdf.xacro (robot description, xacro)
@@ -53,9 +53,25 @@
   <xacro:arg name="initial_positions_file"
     default="$(find tabletop_description)/config/initial_positions.yaml" />
+  <xacro:arg name="base_offset_xyz" default="1.2554 1.0625 0.3085" />
+  <xacro:arg name="base_offset_rpy" default="0.0 0.0 -1.5707" />
+  <xacro:arg name="eef_offset_xyz" default="0.0 0.0 -0.005" />
+  <xacro:arg name="eef_offset_rpy" default="0.0 0.0 0.0" />
+  <xacro:arg name="eef_cylinder_length" default="0.0365" />
+  <xacro:arg name="eef_cylinder_radius" default="0.0315" />
+  <xacro:arg name="eef_cylinder_mass" default="0.5" />
+  <xacro:arg name="eef_sphere_radius" default="0.06" />
   <xacro:property name="initial_positions_file" default="$(arg initial_positions_file)" />
+  <!-- <xacro:arg name="base_offset_xyz" default="1.2468 1.0832 0.2685" /> -->
+  <!-- <xacro:arg name="base_offset_xyz" default="1.2482 1.0588 0.3342" /> -->
+  <!-- <xacro:arg name="base_offset_xyz" default="1.247 1.1279 0.309" /> -->
+  <!-- <xacro:arg name="base_offset_xyz" default="1.2504 1.0625 0.3085" /> -->
+  <!-- <xacro:arg name="bounding_cylinder_radius" default="0.05" />
+    <xacro:arg name="bounding_cylinder_length" default="0.11" /> -->
+  <link name="world" />
   <!-- tabletop -->
-  <xacro:tabletop
+  <xacro:tabletop_robot
     name="$(arg name)"
     tf_prefix="$(arg tf_prefix)"
+    parent="world"
     joint_limits_parameters_file="$(arg joint_limit_params)"
     kinematics_parameters_file="$(arg kinematics_params)"
@@ -66,5 +82,11 @@
     safety_k_position="$(arg safety_k_position)"
     force_abs_paths="$(arg force_abs_paths)"
-  />
+    eef_cylinder_length="$(arg eef_cylinder_length)"
+    eef_cylinder_radius="$(arg eef_cylinder_radius)"
+    eef_cylinder_mass="$(arg eef_cylinder_mass)"
+    eef_sphere_radius="$(arg eef_sphere_radius)">
+    <origin xyz="$(arg base_offset_xyz)" rpy="$(arg base_offset_rpy)" />
+    <origin xyz="$(arg eef_offset_xyz)" rpy="$(arg eef_offset_rpy)" />
+  </xacro:tabletop_robot>
   <xacro:ur_ros2_control
     name="$(arg name)"

File: src/ros/tabletop/tabletop_description/urdf/tabletop_macro.xacro (robot description, xacro)
@@ -3,8 +3,9 @@
   <xacro:include filename="$(find ur_description)/urdf/ur_macro.xacro" />
   <xacro:include filename="$(find tabletop_description)/urdf/eef_macro.xacro" />
-  <xacro:macro name="tabletop"
+  <xacro:macro name="tabletop_robot"
     params="
     name
     tf_prefix
+    parent
     joint_limits_parameters_file
     kinematics_parameters_file
@@ -15,20 +16,16 @@
     safety_k_position
     force_abs_paths
+    eef_cylinder_length
+    eef_cylinder_radius
+    eef_cylinder_mass
+    eef_sphere_radius
+    *origin
+    *eef_origin
     ">
-    <!-- <xacro:property name="robot_offset_xyz" value="1.2468 1.0832 0.2685" /> -->
-    <!-- <xacro:property name="robot_offset_xyz" value="1.2482 1.0588 0.3342" /> -->
-    <!-- <xacro:property name="robot_offset_xyz" value="1.247 1.1279 0.309" /> -->
-    <!-- <xacro:property name="robot_offset_xyz" value="1.2504 1.0625 0.3085" /> -->
-    <xacro:property name="robot_offset_xyz" value="1.2554 1.0625 0.3085" />
-    <xacro:property name="robot_offset_rpy" value="0 0 -1.5707" />
-    <xacro:property name="eef_offset_xyz" value="0 0 -0.005" />
-    <xacro:property name="eef_offset_rpy" value="0 0 0" />
-    <!-- world -->
-    <link name="world" />
     <!-- robot -->
     <xacro:ur_robot
       name="${name}"
       tf_prefix="${tf_prefix}"
-      parent="world"
+      parent="${parent}"
       joint_limits_parameters_file="${joint_limits_parameters_file}"
       kinematics_parameters_file="${kinematics_parameters_file}"
@@ -40,5 +37,5 @@
       force_abs_paths="${force_abs_paths}"
     >
-      <origin xyz="${robot_offset_xyz}" rpy="${robot_offset_rpy}" />
+      <xacro:insert_block name="origin" />
     </xacro:ur_robot>
     <!-- end effector -->
@@ -46,6 +43,10 @@
       tf_prefix="${tf_prefix}"
       parent="${tf_prefix}wrist_3_link"
+      cylinder_length="${eef_cylinder_length}"
+      cylinder_radius="${eef_cylinder_radius}"
+      cylinder_mass="${eef_cylinder_mass}"
+      sphere_radius="${eef_sphere_radius}"
     >
-      <origin xyz="${eef_offset_xyz}" rpy="${eef_offset_rpy}" />
+      <xacro:insert_block name="eef_origin" />
     </xacro:eef>
   </xacro:macro>

Commit message: I think I found the right position

File: src/ros/tabletop/tabletop_description/urdf/eef_macro.xacro (robot description, xacro)
@@ -7,9 +7,9 @@
     tf_prefix
     parent
-    *origin
     cylinder_length
     cylinder_radius
     cylinder_mass
     sphere_radius
+    *origin
     ">
     <link name="${tf_prefix}eef_link">

File: src/ros/tabletop/tabletop_description/urdf/sphere_macro.xacro (robot description, xacro)
@@ -6,6 +6,6 @@
     tf_prefix
     parent
+    radius
     *origin
-    radius
     ">
     <link name="${tf_prefix}${name}">

File: src/ros/tabletop/tabletop_description/urdf/tabletop.urdf.xacro (robot description, xacro)
@@ -53,17 +53,17 @@
   <xacro:arg name="initial_positions_file"
     default="$(find tabletop_description)/config/initial_positions.yaml" />
-  <xacro:arg name="base_offset_xyz" default="1.2554 1.0625 0.3085" />
-  <xacro:arg name="base_offset_rpy" default="0.0 0.0 -1.5707" />
-  <xacro:arg name="eef_offset_xyz" default="0.0 0.0 -0.005" />
-  <xacro:arg name="eef_offset_rpy" default="0.0 0.0 0.0" />
+  <xacro:property name="initial_positions_file" default="$(arg initial_positions_file)" />
   <xacro:arg name="eef_cylinder_length" default="0.0365" />
   <xacro:arg name="eef_cylinder_radius" default="0.0315" />
   <xacro:arg name="eef_cylinder_mass" default="0.5" />
   <xacro:arg name="eef_sphere_radius" default="0.06" />
-  <xacro:property name="initial_positions_file" default="$(arg initial_positions_file)" />
-  <!-- <xacro:arg name="base_offset_xyz" default="1.2468 1.0832 0.2685" /> -->
-  <!-- <xacro:arg name="base_offset_xyz" default="1.2482 1.0588 0.3342" /> -->
-  <!-- <xacro:arg name="base_offset_xyz" default="1.247 1.1279 0.309" /> -->
-  <!-- <xacro:arg name="base_offset_xyz" default="1.2504 1.0625 0.3085" /> -->
+  <xacro:arg name="eef_origin_xyz" default="0.0 0.0 -0.005" />
+  <xacro:arg name="eef_origin_rpy" default="0.0 0.0 0.0" />
+  <xacro:arg name="base_origin_xyz" default="0.0 0.0 0.0" />
+  <xacro:arg name="base_origin_rpy" default="0.0 0.0 0.0" />
+  <!-- <xacro:arg name="base_origin_xyz" default="1.2468 1.0832 0.2685" /> -->
+  <!-- <xacro:arg name="base_origin_xyz" default="1.2482 1.0588 0.3342" /> -->
+  <!-- <xacro:arg name="base_origin_xyz" default="1.247 1.1279 0.309" /> -->
+  <!-- <xacro:arg name="base_origin_xyz" default="1.2504 1.0625 0.3085" /> -->
   <!-- <xacro:arg name="bounding_cylinder_radius" default="0.05" />
     <xacro:arg name="bounding_cylinder_length" default="0.11" /> -->
@@ -86,6 +86,6 @@
     eef_cylinder_mass="$(arg eef_cylinder_mass)"
     eef_sphere_radius="$(arg eef_sphere_radius)">
-    <origin xyz="$(arg base_offset_xyz)" rpy="$(arg base_offset_rpy)" />
-    <origin xyz="$(arg eef_offset_xyz)" rpy="$(arg eef_offset_rpy)" />
+    <origin xyz="$(arg base_origin_xyz)" rpy="$(arg base_origin_rpy)" />
+    <origin xyz="$(arg eef_origin_xyz)" rpy="$(arg eef_origin_rpy)" />
   </xacro:tabletop_robot>
   <xacro:ur_ros2_control

Commit message: Simplified tabletop_description

File: src/ros/tabletop/tabletop_description/urdf/eef_macro.xacro (robot description, xacro)
@@ -1,6 +1,4 @@
 <?xml version="1.0"?>
 <robot xmlns:xacro="http://ros.org/wiki/xacro">
-  <xacro:include filename="$(find tabletop_description)/urdf/sphere_macro.xacro" />
-  <xacro:include filename="$(find tabletop_description)/urdf/cylinder_macro.xacro" />
   <xacro:macro name="eef"
     params="
@@ -40,16 +38,21 @@
       </inertial>
     </link>
-    <xacro:sphere
-      name="eef_sphere"
-      tf_prefix="${tf_prefix}"
-      parent="${parent}"
-      radius="${sphere_radius}"
-    >
-      <xacro:insert_block name="origin" />
-    </xacro:sphere>
-    <joint name="${parent}-eef_link" type="fixed">
+    <link name="${tf_prefix}eef_sphere">
+      <collision>
+        <geometry>
+          <sphere radius="${sphere_radius}" />
+        </geometry>
+        <origin rpy="0 0 0" xyz="0 0 0" />
+      </collision>
+    </link>
+    <joint name="${tf_prefix}${parent}-eef_link" type="fixed">
       <xacro:insert_block name="origin" />
       <parent link="${parent}" />
       <child link="${tf_prefix}eef_link" />
+    </joint>
+    <joint name="${tf_prefix}${parent}-eef_sphere" type="fixed">
+      <xacro:insert_block name="origin" />
+      <parent link="${parent}" />
+      <child link="${tf_prefix}eef_sphere" />
     </joint>
     <!-- eef frame, X+ direction to move to attach object,
@@ -62,13 +65,4 @@
       <child link="${tf_prefix}eef" />
     </joint>
-    <!-- <xacro:cylinder
-      name="bounding_cylinder"
-      tf_prefix="${tf_prefix}"
-      parent="${tf_prefix}eef"
-      radius="${bounding_cylinder_radius}"
-      length="${bounding_cylinder_length}"
-    >
-      <origin xyz="0 0 0" rpy="0 0 0" />
-    </xacro:cylinder> -->
   </xacro:macro>
 </robot>

File: src/ros/tabletop/tabletop_description/urdf/tabletop.urdf.xacro (robot description, xacro)
@@ -54,4 +54,5 @@
     default="$(find tabletop_description)/config/initial_positions.yaml" />
   <xacro:property name="initial_positions_file" default="$(arg initial_positions_file)" />
+  <!-- end-effector paramaters -->
   <xacro:arg name="eef_cylinder_length" default="0.0365" />
   <xacro:arg name="eef_cylinder_radius" default="0.0315" />
@@ -60,12 +61,7 @@
   <xacro:arg name="eef_origin_xyz" default="0.0 0.0 -0.005" />
   <xacro:arg name="eef_origin_rpy" default="0.0 0.0 0.0" />
+  <!-- base parameters -->
   <xacro:arg name="base_origin_xyz" default="0.0 0.0 0.0" />
   <xacro:arg name="base_origin_rpy" default="0.0 0.0 0.0" />
-  <!-- <xacro:arg name="base_origin_xyz" default="1.2468 1.0832 0.2685" /> -->
-  <!-- <xacro:arg name="base_origin_xyz" default="1.2482 1.0588 0.3342" /> -->
-  <!-- <xacro:arg name="base_origin_xyz" default="1.247 1.1279 0.309" /> -->
-  <!-- <xacro:arg name="base_origin_xyz" default="1.2504 1.0625 0.3085" /> -->
-  <!-- <xacro:arg name="bounding_cylinder_radius" default="0.05" />
-    <xacro:arg name="bounding_cylinder_length" default="0.11" /> -->
   <link name="world" />
   <!-- tabletop -->

Commit message: huh

File: src/ros/tabletop/tabletop_description/urdf/eef_macro.xacro (robot description, xacro)
@@ -17,6 +17,6 @@
         </geometry>
         <origin xyz="0 0 0" rpy="0 0 0" />
-        <material name="black">
-          <color rgba="0 0 0 1" />
+        <material name="dark_gray">
+          <color rgba="0.2 0.2 0.2 1" />
         </material>
       </visual>

File: src/ros/tabletop/tabletop_moveit_config/srdf/dual_tabletop_macro.srdf.xacro (robot description, xacro)
@@ -50,10 +50,10 @@
     </group_state>
     <group_state name="present" group="left_manipulator">
-      <joint name="left_shoulder_pan_joint" value="1.1485" />
-      <joint name="left_shoulder_lift_joint" value="-2.4295" />
-      <joint name="left_elbow_joint" value="-1.5077" />
-      <joint name="left_wrist_1_joint" value="-0.7742" />
-      <joint name="left_wrist_2_joint" value="-1.5707" />
-      <joint name="left_wrist_3_joint" value="2.5884" />
+      <joint name="left_shoulder_pan_joint" value="1.1109" />
+      <joint name="left_shoulder_lift_joint" value="-2.1167" />
+      <joint name="left_elbow_joint" value="-2.2282" />
+      <joint name="left_wrist_1_joint" value="-0.3597" />
+      <joint name="left_wrist_2_joint" value="-1.5763" />
+      <joint name="left_wrist_3_joint" value="2.0311" />
     </group_state>
     <group_state name="test_object_attached" group="left_manipulator">
@@ -80,13 +80,13 @@
       <joint name="right_wrist_1_joint" value="${-pi/3}" />
       <joint name="right_wrist_2_joint" value="${pi/2}" />
-      <joint name="right_wrist_3_joint" value="${pi}" />
+      <joint name="right_wrist_3_joint" value="${-pi}" />
     </group_state>
     <group_state name="present" group="right_manipulator">
-      <joint name="right_shoulder_pan_joint" value="-0.6065" />
-      <joint name="right_shoulder_lift_joint" value="-0.6788" />
-      <joint name="right_elbow_joint" value="1.4381" />
-      <joint name="right_wrist_1_joint" value="-2.3351" />
+      <joint name="right_shoulder_pan_joint" value="-1.1504" />
+      <joint name="right_shoulder_lift_joint" value="-0.9975" />
+      <joint name="right_elbow_joint" value="2.1476" />
+      <joint name="right_wrist_1_joint" value="-2.7118" />
       <joint name="right_wrist_2_joint" value="1.5686" />
-      <joint name="right_wrist_3_joint" value="3.7411" />
+      <joint name="right_wrist_3_joint" value="-1.9871" />
     </group_state>
     <group_state name="test_object_attached" group="right_manipulator">
