Commit message: Working smoothly again, took a whirl at state machines, it's not worth it

File: src/ros/tabletop/tabletop_moveit_config/srdf/tabletop_macro.srdf.xacro (robot description, xacro)
@@ -62,5 +62,5 @@
       <joint name="wrist_3_joint" value="${pi}" />
     </group_state>
-    <group_state name="pre_present" group="manipulator">
+    <group_state name="present" group="manipulator">
       <joint name="shoulder_pan_joint" value="-0.6065" />
       <joint name="shoulder_lift_joint" value="-0.6788" />
@@ -69,4 +69,12 @@
       <joint name="wrist_2_joint" value="1.5686" />
       <joint name="wrist_3_joint" value="3.7411" />
+    </group_state>
+    <group_state name="fetched" group="manipulator">
+      <joint name="shoulder_pan_joint" value="-0.2" />
+      <joint name="shoulder_lift_joint" value="${-pi/2}" />
+      <joint name="elbow_joint" value="${pi/2}" />
+      <joint name="wrist_1_joint" value="${-pi/2}" />
+      <joint name="wrist_2_joint" value="${pi/2}" />
+      <joint name="wrist_3_joint" value="${pi}" />
     </group_state>
     <!--VIRTUAL

Commit message: State machine seems to be working?

File: src/ros/tabletop/tabletop_moveit_config/srdf/tabletop_macro.srdf.xacro (robot description, xacro)
@@ -78,4 +78,12 @@
       <joint name="wrist_3_joint" value="${pi}" />
     </group_state>
+    <group_state name="test_object_attached" group="manipulator">
+      <joint name="shoulder_pan_joint" value="-0.2" />
+      <joint name="shoulder_lift_joint" value="${-pi/2}" />
+      <joint name="elbow_joint" value="${pi/2}" />
+      <joint name="wrist_1_joint" value="${-pi/2}" />
+      <joint name="wrist_2_joint" value="${pi}" />
+      <joint name="wrist_3_joint" value="${pi}" />
+    </group_state>
     <!--VIRTUAL
     JOINT - Purpose - this element defines a virtual joint between a robot link and an external

Commit message: Object attached detection implemented, smooth pursuit updated, smooth pursuit object and test object stls added

File: src/ros/tabletop/tabletop_moveit_config/srdf/tabletop_macro.srdf.xacro (robot description, xacro)
@@ -79,9 +79,9 @@
     </group_state>
     <group_state name="test_object_attached" group="manipulator">
-      <joint name="shoulder_pan_joint" value="-0.2" />
+      <joint name="shoulder_pan_joint" value="${-pi/2}" />
       <joint name="shoulder_lift_joint" value="${-pi/2}" />
       <joint name="elbow_joint" value="${pi/2}" />
       <joint name="wrist_1_joint" value="${-pi/2}" />
-      <joint name="wrist_2_joint" value="${pi}" />
+      <joint name="wrist_2_joint" value="0" />
       <joint name="wrist_3_joint" value="${pi}" />
     </group_state>
