Commit message: Working on two robots

File: src/ros/tabletop/tabletop_moveit_config/srdf/dual_tabletop_macro.srdf.xacro (robot description, xacro)
@@ -30,5 +30,6 @@
       <chain base_link="right_base_link" tip_link="right_eef" />
     </group>
-    <!--GROUP STATES -->
+    <!--GROUP
+    STATES -->
     <!-- Left arm group states -->
     <group_state name="erect" group="left_manipulator">
@@ -73,5 +74,5 @@
     </group_state>
     <group_state name="fetched" group="left_manipulator">
-      <joint name="left_shoulder_pan_joint" value="-0.2" />
+      <joint name="left_shoulder_pan_joint" value="0.2" />
       <joint name="left_shoulder_lift_joint" value="${-pi/2}" />
       <joint name="left_elbow_joint" value="${pi/2}" />
@@ -81,5 +82,5 @@
     </group_state>
     <group_state name="test_object_attached" group="left_manipulator">
-      <joint name="left_shoulder_pan_joint" value="${-pi/2}" />
+      <joint name="left_shoulder_pan_joint" value="${-pi/4}" />
       <joint name="left_shoulder_lift_joint" value="${-pi/2}" />
       <joint name="left_elbow_joint" value="${pi/2}" />
@@ -138,5 +139,5 @@
     </group_state>
     <group_state name="test_object_attached" group="right_manipulator">
-      <joint name="right_shoulder_pan_joint" value="${-pi/2}" />
+      <joint name="right_shoulder_pan_joint" value="${-pi/6}" />
       <joint name="right_shoulder_lift_joint" value="${-pi/2}" />
       <joint name="right_elbow_joint" value="${pi/2}" />
@@ -145,8 +146,12 @@
       <joint name="right_wrist_3_joint" value="${pi}" />
     </group_state>
-    <!--VIRTUAL JOINTS -->
-    <virtual_joint name="left_virtual_joint" type="fixed" parent_frame="world" child_link="left_base_link" />
-    <virtual_joint name="right_virtual_joint" type="fixed" parent_frame="world" child_link="right_base_link" />
-    <!--DISABLE COLLISIONS -->
+    <!--VIRTUAL
+    JOINTS -->
+    <virtual_joint name="left_virtual_joint" type="fixed" parent_frame="world"
+      child_link="left_base_link" />
+    <virtual_joint name="right_virtual_joint" type="fixed" parent_frame="world"
+      child_link="right_base_link" />
+    <!--DISABLE
+    COLLISIONS -->
     <!-- Left arm collisions -->
     <disable_collisions link1="left_base_link_inertia" link2="left_shoulder_link" reason="Adjacent" />
@@ -166,5 +171,6 @@
     <disable_collisions link1="left_eef_link" link2="left_eef_sphere" reason="Default" />
     <!-- Right arm collisions -->
-    <disable_collisions link1="right_base_link_inertia" link2="right_shoulder_link" reason="Adjacent" />
+    <disable_collisions link1="right_base_link_inertia" link2="right_shoulder_link"
+      reason="Adjacent" />
     <disable_collisions link1="right_shoulder_link" link2="right_upper_arm_link" reason="Adjacent" />
     <disable_collisions link1="right_upper_arm_link" link2="right_forearm_link" reason="Adjacent" />

Commit message: we must imagine sisyphus happy

File: src/ros/tabletop/tabletop_moveit_config/srdf/dual_tabletop_macro.srdf.xacro (robot description, xacro)
@@ -66,13 +66,13 @@
     </group_state>
     <group_state name="present" group="left_manipulator">
-      <joint name="left_shoulder_pan_joint" value="-0.6065" />
-      <joint name="left_shoulder_lift_joint" value="-0.6788" />
-      <joint name="left_elbow_joint" value="1.4381" />
-      <joint name="left_wrist_1_joint" value="-2.3351" />
-      <joint name="left_wrist_2_joint" value="1.5686" />
-      <joint name="left_wrist_3_joint" value="3.7411" />
+      <joint name="left_shoulder_pan_joint" value="0.1734" />
+      <joint name="left_shoulder_lift_joint" value="-0.7113" />
+      <joint name="left_elbow_joint" value="1.5066" />
+      <joint name="left_wrist_1_joint" value="-2.3671" />
+      <joint name="left_wrist_2_joint" value="1.5707" />
+      <joint name="left_wrist_3_joint" value="2.9664" />
     </group_state>
     <group_state name="fetched" group="left_manipulator">
-      <joint name="left_shoulder_pan_joint" value="0.2" />
+      <joint name="left_shoulder_pan_joint" value="-0.2" />
       <joint name="left_shoulder_lift_joint" value="${-pi/2}" />
       <joint name="left_elbow_joint" value="${pi/2}" />

Commit message: Reckless abandon

File: src/ros/tabletop/tabletop_moveit_config/srdf/dual_tabletop_macro.srdf.xacro (robot description, xacro)
@@ -33,51 +33,27 @@
     STATES -->
     <!-- Left arm group states -->
-    <group_state name="erect" group="left_manipulator">
-      <joint name="left_shoulder_pan_joint" value="0" />
-      <joint name="left_shoulder_lift_joint" value="${-pi/2}" />
-      <joint name="left_elbow_joint" value="0" />
-      <joint name="left_wrist_1_joint" value="0" />
-      <joint name="left_wrist_2_joint" value="0" />
-      <joint name="left_wrist_3_joint" value="0" />
-    </group_state>
-    <group_state name="flaccid" group="left_manipulator">
-      <joint name="left_shoulder_pan_joint" value="0" />
-      <joint name="left_shoulder_lift_joint" value="0" />
-      <joint name="left_elbow_joint" value="0" />
-      <joint name="left_wrist_1_joint" value="0" />
-      <joint name="left_wrist_2_joint" value="0" />
-      <joint name="left_wrist_3_joint" value="0" />
-    </group_state>
-    <group_state name="semi" group="left_manipulator">
-      <joint name="left_shoulder_pan_joint" value="0" />
-      <joint name="left_shoulder_lift_joint" value="${-pi/2}" />
-      <joint name="left_elbow_joint" value="${pi/2}" />
-      <joint name="left_wrist_1_joint" value="${-pi/2}" />
-      <joint name="left_wrist_2_joint" value="0" />
-      <joint name="left_wrist_3_joint" value="0" />
-    </group_state>
     <group_state name="idle" group="left_manipulator">
       <joint name="left_shoulder_pan_joint" value="0" />
-      <joint name="left_shoulder_lift_joint" value="${-5*pi/6}" />
-      <joint name="left_elbow_joint" value="${2*pi/3}" />
-      <joint name="left_wrist_1_joint" value="${-pi/3}" />
-      <joint name="left_wrist_2_joint" value="${pi/2}" />
+      <joint name="left_shoulder_lift_joint" value="${-pi/6}" />
+      <joint name="left_elbow_joint" value="${-2*pi/3}" />
+      <joint name="left_wrist_1_joint" value="${-2*pi/3}" />
+      <joint name="left_wrist_2_joint" value="${-pi/2}" />
+      <joint name="left_wrist_3_joint" value="${pi}" />
+    </group_state>
+    <group_state name="fetched" group="left_manipulator">
+      <joint name="left_shoulder_pan_joint" value="0.2" />
+      <joint name="left_shoulder_lift_joint" value="${-pi/2}" />
+      <joint name="left_elbow_joint" value="${-pi/2}" />
+      <joint name="left_wrist_1_joint" value="${-pi/2}" />
+      <joint name="left_wrist_2_joint" value="${-pi/2}" />
       <joint name="left_wrist_3_joint" value="${pi}" />
     </group_state>
     <group_state name="present" group="left_manipulator">
-      <joint name="left_shoulder_pan_joint" value="0.1734" />
-      <joint name="left_shoulder_lift_joint" value="-0.7113" />
-      <joint name="left_elbow_joint" value="1.5066" />
-      <joint name="left_wrist_1_joint" value="-2.3671" />
-      <joint name="left_wrist_2_joint" value="1.5707" />
-      <joint name="left_wrist_3_joint" value="2.9664" />
-    </group_state>
-    <group_state name="fetched" group="left_manipulator">
-      <joint name="left_shoulder_pan_joint" value="-0.2" />
-      <joint name="left_shoulder_lift_joint" value="${-pi/2}" />
-      <joint name="left_elbow_joint" value="${pi/2}" />
-      <joint name="left_wrist_1_joint" value="${-pi/2}" />
-      <joint name="left_wrist_2_joint" value="${pi/2}" />
-      <joint name="left_wrist_3_joint" value="${pi}" />
+      <joint name="left_shoulder_pan_joint" value="0.553" />
+      <joint name="left_shoulder_lift_joint" value="-2.4295" />
+      <joint name="left_elbow_joint" value="-1.5077" />
+      <joint name="left_wrist_1_joint" value="-0.7742" />
+      <joint name="left_wrist_2_joint" value="-1.5707" />
+      <joint name="left_wrist_3_joint" value="2.5884" />
     </group_state>
     <group_state name="test_object_attached" group="left_manipulator">
@@ -90,28 +66,4 @@
     </group_state>
     <!-- Right arm group states -->
-    <group_state name="erect" group="right_manipulator">
-      <joint name="right_shoulder_pan_joint" value="0" />
-      <joint name="right_shoulder_lift_joint" value="${-pi/2}" />
-      <joint name="right_elbow_joint" value="0" />
-      <joint name="right_wrist_1_joint" value="0" />
-      <joint name="right_wrist_2_joint" value="0" />
-      <joint name="right_wrist_3_joint" value="0" />
-    </group_state>
-    <group_state name="flaccid" group="right_manipulator">
-      <joint name="right_shoulder_pan_joint" value="0" />
-      <joint name="right_shoulder_lift_joint" value="0" />
-      <joint name="right_elbow_joint" value="0" />
-      <joint name="right_wrist_1_joint" value="0" />
-      <joint name="right_wrist_2_joint" value="0" />
-      <joint name="right_wrist_3_joint" value="0" />
-    </group_state>
-    <group_state name="semi" group="right_manipulator">
-      <joint name="right_shoulder_pan_joint" value="0" />
-      <joint name="right_shoulder_lift_joint" value="${-pi/2}" />
-      <joint name="right_elbow_joint" value="${pi/2}" />
-      <joint name="right_wrist_1_joint" value="${-pi/2}" />
-      <joint name="right_wrist_2_joint" value="0" />
-      <joint name="right_wrist_3_joint" value="0" />
-    </group_state>
     <group_state name="idle" group="right_manipulator">
       <joint name="right_shoulder_pan_joint" value="0" />
@@ -119,4 +71,12 @@
       <joint name="right_elbow_joint" value="${2*pi/3}" />
       <joint name="right_wrist_1_joint" value="${-pi/3}" />
+      <joint name="right_wrist_2_joint" value="${pi/2}" />
+      <joint name="right_wrist_3_joint" value="${pi}" />
+    </group_state>
+    <group_state name="fetched" group="right_manipulator">
+      <joint name="right_shoulder_pan_joint" value="-0.2" />
+      <joint name="right_shoulder_lift_joint" value="${-pi/2}" />
+      <joint name="right_elbow_joint" value="${pi/2}" />
+      <joint name="right_wrist_1_joint" value="${-pi/2}" />
       <joint name="right_wrist_2_joint" value="${pi/2}" />
       <joint name="right_wrist_3_joint" value="${pi}" />
@@ -129,12 +89,4 @@
       <joint name="right_wrist_2_joint" value="1.5686" />
       <joint name="right_wrist_3_joint" value="3.7411" />
-    </group_state>
-    <group_state name="fetched" group="right_manipulator">
-      <joint name="right_shoulder_pan_joint" value="-0.2" />
-      <joint name="right_shoulder_lift_joint" value="${-pi/2}" />
-      <joint name="right_elbow_joint" value="${pi/2}" />
-      <joint name="right_wrist_1_joint" value="${-pi/2}" />
-      <joint name="right_wrist_2_joint" value="${pi/2}" />
-      <joint name="right_wrist_3_joint" value="${pi}" />
     </group_state>
     <group_state name="test_object_attached" group="right_manipulator">

Commit message: Modified rig file

File: src/ros/tabletop/tabletop_moveit_config/srdf/dual_tabletop_macro.srdf.xacro (robot description, xacro)
@@ -42,13 +42,13 @@
     </group_state>
     <group_state name="fetched" group="left_manipulator">
-      <joint name="left_shoulder_pan_joint" value="0.2" />
-      <joint name="left_shoulder_lift_joint" value="${-pi/2}" />
-      <joint name="left_elbow_joint" value="${-pi/2}" />
-      <joint name="left_wrist_1_joint" value="${-pi/2}" />
+      <joint name="left_shoulder_pan_joint" value="0" />
+      <joint name="left_shoulder_lift_joint" value="${-pi/6}" />
+      <joint name="left_elbow_joint" value="${-2*pi/3}" />
+      <joint name="left_wrist_1_joint" value="${-2*pi/3}" />
       <joint name="left_wrist_2_joint" value="${-pi/2}" />
       <joint name="left_wrist_3_joint" value="${pi}" />
     </group_state>
     <group_state name="present" group="left_manipulator">
-      <joint name="left_shoulder_pan_joint" value="0.553" />
+      <joint name="left_shoulder_pan_joint" value="1.1485" />
       <joint name="left_shoulder_lift_joint" value="-2.4295" />
       <joint name="left_elbow_joint" value="-1.5077" />
@@ -75,8 +75,8 @@
     </group_state>
     <group_state name="fetched" group="right_manipulator">
-      <joint name="right_shoulder_pan_joint" value="-0.2" />
-      <joint name="right_shoulder_lift_joint" value="${-pi/2}" />
-      <joint name="right_elbow_joint" value="${pi/2}" />
-      <joint name="right_wrist_1_joint" value="${-pi/2}" />
+      <joint name="right_shoulder_pan_joint" value="0" />
+      <joint name="right_shoulder_lift_joint" value="${-5*pi/6}" />
+      <joint name="right_elbow_joint" value="${2*pi/3}" />
+      <joint name="right_wrist_1_joint" value="${-pi/3}" />
       <joint name="right_wrist_2_joint" value="${pi/2}" />
       <joint name="right_wrist_3_joint" value="${pi}" />

Commit message: wtf am I doing

File: src/ros/tabletop/tabletop_moveit_config/srdf/dual_tabletop_macro.srdf.xacro (robot description, xacro)
@@ -34,10 +34,10 @@
     <!-- Left arm group states -->
     <group_state name="idle" group="left_manipulator">
-      <joint name="left_shoulder_pan_joint" value="0" />
-      <joint name="left_shoulder_lift_joint" value="${-pi/6}" />
-      <joint name="left_elbow_joint" value="${-2*pi/3}" />
-      <joint name="left_wrist_1_joint" value="${-2*pi/3}" />
-      <joint name="left_wrist_2_joint" value="${-pi/2}" />
-      <joint name="left_wrist_3_joint" value="${pi}" />
+      <joint name="left_shoulder_pan_joint" value="0.0" />
+      <joint name="left_shoulder_lift_joint" value="${-pi/2}" />
+      <joint name="left_elbow_joint" value="${pi/2}" />
+      <joint name="left_wrist_1_joint" value="${-pi/2}" />
+      <joint name="left_wrist_2_joint" value="${pi/2}" />
+      <joint name="left_wrist_3_joint" value="0.0" />
     </group_state>
     <group_state name="fetched" group="left_manipulator">
@@ -67,10 +67,10 @@
     <!-- Right arm group states -->
     <group_state name="idle" group="right_manipulator">
-      <joint name="right_shoulder_pan_joint" value="0" />
-      <joint name="right_shoulder_lift_joint" value="${-5*pi/6}" />
-      <joint name="right_elbow_joint" value="${2*pi/3}" />
-      <joint name="right_wrist_1_joint" value="${-pi/3}" />
-      <joint name="right_wrist_2_joint" value="${pi/2}" />
-      <joint name="right_wrist_3_joint" value="${pi}" />
+      <joint name="right_shoulder_pan_joint" value="0.0" />
+      <joint name="right_shoulder_lift_joint" value="${-pi/2}" />
+      <joint name="right_elbow_joint" value="${-pi/2}" />
+      <joint name="right_wrist_1_joint" value="${-pi/2}" />
+      <joint name="right_wrist_2_joint" value="${-pi/2}" />
+      <joint name="right_wrist_3_joint" value="0.0" />
     </group_state>
     <group_state name="fetched" group="right_manipulator">
@@ -98,4 +98,26 @@
       <joint name="right_wrist_3_joint" value="${pi}" />
     </group_state>
+    <!--JOINT
+    PROPERTIES - Per-joint weights applied to the path-length distance metric used by
+    JointModelGroup::distance(), and therefore by OMPL's PathLengthOptimizationObjective.
+    Higher value = joint contributes more to path cost = planner prefers to move it less.
+    Bias here penalizes proximal motion to keep the base/shoulder steadier and let the
+    wrist do more of the work. -->
+    <joint_property joint_name="left_shoulder_pan_joint" property_name="distance_factor"
+      value="4.0" />
+    <joint_property joint_name="left_shoulder_lift_joint" property_name="distance_factor"
+      value="3.0" />
+    <joint_property joint_name="left_elbow_joint" property_name="distance_factor" value="2.0" />
+    <joint_property joint_name="left_wrist_1_joint" property_name="distance_factor" value="1.0" />
+    <joint_property joint_name="left_wrist_2_joint" property_name="distance_factor" value="1.0" />
+    <joint_property joint_name="left_wrist_3_joint" property_name="distance_factor" value="1.0" />
+    <joint_property joint_name="right_shoulder_pan_joint" property_name="distance_factor"
+      value="4.0" />
+    <joint_property joint_name="right_shoulder_lift_joint" property_name="distance_factor"
+      value="3.0" />
+    <joint_property joint_name="right_elbow_joint" property_name="distance_factor" value="2.0" />
+    <joint_property joint_name="right_wrist_1_joint" property_name="distance_factor" value="1.0" />
+    <joint_property joint_name="right_wrist_2_joint" property_name="distance_factor" value="1.0" />
+    <joint_property joint_name="right_wrist_3_joint" property_name="distance_factor" value="1.0" />
     <!--VIRTUAL
     JOINTS -->
